Commit message: first update

File: urdf/akros2.urdf (robot description, URDF)
Before this commit: robot akros, 10 links, 9 joints
Links:
- added link nav_link, mass 0.001; collision box size=0.21 0.15 0.099; visual mesh filename=package://akros2_description/meshes/navigation_module.stl
- link base_footprint: mass 1.0 -> None; geometry collision box size=0.21 0.24 0.18
- link base_link: geometry collision box size=0.21 0.15 0.045; visual mesh filename=package://akros2_description/meshes/base_module.stl
- link base_link_inertial: mass 0.001 -> 1.0
- link laser_link: geometry collision mesh filename=package://akros2_description/meshes/ld06.stl; visual mesh filename=package://akros2_description/meshes/ld06.stl
Joints:
- removed joint base_lidar_fixed
- removed joint base_link_footprint_fixed
- removed joint base_t265_fixed
- added joint base_footprint_fixed: type fixed, parent base_link, child base_footprint, origin xyz=0 0 0
- added joint base_link_nav_fixed: type fixed, parent base_link, child nav_link, origin xyz=0 0 0.099, axis 0 0 0
- added joint nav_laser_fixed: type fixed, parent nav_link, child laser_link, origin xyz=0.0632 0 0.0155
- added joint nav_t265_fixed: type fixed, parent nav_link, child t265_pose_frame, origin xyz=0.094 0 0.016 rpy=0 0 0
- joint base_inertial_fixed: origin xyz=0 0 0 rpy=0 0 0 -> xyz=0 0 0
- joint laser_frame_fixed: origin xyz=0 0 0.03 rpy=0 0 0 -> xyz=0 0 0.0255

Commit message: updated description

File: urdf/akros2.urdf (robot description, URDF)
Before this commit: robot akros, 11 links, 10 joints
Links:
- added link t265_pose_inertial, mass 0.1
- link t265_pose_frame: mass 0.1 -> None
Joints:
- removed joint base_link_nav_fixed
- removed joint nav_t265_fixed
- added joint base_nav_fixed: type fixed, parent base_link, child nav_link, origin xyz=0 0 0.099, axis 0 0 0
- added joint pose_base_fixed: type fixed, parent t265_pose_frame, child base_link, origin xyz=-0.094 0 -0.115
- added joint pose_inertial_fixed: type fixed, parent t265_pose_frame, child t265_pose_inertial, origin xyz=0 0 0

Commit message: update URDF

File: urdf/akros2.urdf (robot description, URDF)
Before this commit: robot akros, 12 links, 11 joints
Links:
- link base_footprint: geometry 

Commit message: updated urdf

File: urdf/akros2.urdf (robot description, URDF)
Before this commit: robot akros, 12 links, 11 joints
Links:
- link base_link: geometry collision mesh filename=package://akros2_description/meshes/base_module.stl; visual mesh filename=package://akros2_description/meshes/base_module.stl
- link nav_link: geometry collision mesh filename=package://akros2_description/meshes/navigation_module.stl; visual mesh filename=package://akros2_description/meshes/navigation_module.stl
- link t265_pose_frame: geometry collision mesh filename=package://akros2_description/meshes/t265.stl; visual mesh filename=package://akros2_description/meshes/t265.stl
- link wheel_lb: geometry collision mesh filename=package://akros2_description/meshes/wheel_lb.stl; visual mesh filename=package://akros2_description/meshes/wheel_lb.stl
- link wheel_lf: geometry collision mesh filename=package://akros2_description/meshes/wheel_lf.stl; visual mesh filename=package://akros2_description/meshes/wheel_lf.stl
- link wheel_rb: geometry collision mesh filename=package://akros2_description/meshes/wheel_rb.stl; visual mesh filename=package://akros2_description/meshes/wheel_rb.stl
- link wheel_rf: geometry collision mesh filename=package://akros2_description/meshes/wheel_rf.stl; visual mesh filename=package://akros2_description/meshes/wheel_rf.stl

Commit message: update meshes from stl to dae

File: urdf/akros2.urdf (robot description, URDF)
Before this commit: robot akros, 12 links, 11 joints
Links:
- added link imu_frame
- added link imu_link
- link base_link: geometry collision mesh filename=package://akros2_description/meshes/base_module.dae; visual mesh filename=package://akros2_description/meshes/base_module.dae
- link laser_link: geometry collision mesh filename=package://akros2_description/meshes/ld06.dae; visual mesh filename=package://akros2_description/meshes/ld06.dae
- link nav_link: geometry collision mesh filename=package://akros2_description/meshes/navigation_module.dae; visual mesh filename=package://akros2_description/meshes/navigation_module.dae
- link t265_pose_frame: geometry collision mesh filename=package://akros2_description/meshes/t265.dae; visual mesh filename=package://akros2_description/meshes/t265.dae
- link wheel_lb: geometry collision cylinder length=0.035 radius=0.04; visual mesh filename=package://akros2_description/meshes/wheel_lb.dae
- link wheel_lf: geometry collision cylinder length=0.035 radius=0.04; visual mesh filename=package://akros2_description/meshes/wheel_lf.dae
- link wheel_rb: geometry collision cylinder length=0.035 radius=0.04; visual mesh filename=package://akros2_description/meshes/wheel_rb.dae
- link wheel_rf: geometry collision cylinder length=0.035 radius=0.04; visual mesh filename=package://akros2_description/meshes/wheel_rf.dae
Joints:
- added joint imu_base_fixed: type fixed, parent base_link, child imu_link, origin xyz=0 0 0
- added joint imu_frame_fixed: type fixed, parent imu_link, child imu_frame, origin xyz=0 0 0
