Commit message: update urdf geometries, .urdf to .xacro

File: urdf/akros2.urdf.xacro (robot description, xacro)
@@ -27,4 +27,5 @@
     <origin xyz="0 0 0.0278" rpy="0 0 0" />
     <geometry>
+      <box size="0.210 0.174 0.037"/>
       <mesh filename="package://akros2_description/meshes/base_module.dae" />
     </geometry>
@@ -35,5 +36,5 @@
   <inertial>
     <origin xyz="0 0 0" rpy="0 0 0" />
-    <mass value="1.0"/>
+    <mass value="2.0"/>
     <inertia ixx="0.015" iyy="0.0375" izz="0.0375" ixy="0" ixz="0" iyz="0"/>
   </inertial>
@@ -44,5 +45,5 @@
 <link name="nav_link">
   <inertial>
-    <mass value="0.001" />
+    <mass value="0.5" />
     <inertia ixx="0.01" ixy="0.01" ixz="0.01" iyy="0.01" iyz="0.01" izz="0.01" />
   </inertial>
@@ -57,4 +58,5 @@
     <origin xyz="0 0 -0.099" rpy="0 0 0" />
     <geometry>
+      <box size="0.2 0.154 0.037"/>
       <mesh filename="package://akros2_description/meshes/navigation_module.dae" />
     </geometry>
@@ -65,5 +67,5 @@
   <inertial>
     <origin xyz="0 0 0" rpy="0 0 0" />
-    <mass value="0.001" />
+    <mass value="0.12" />
     <inertia ixx="0.01" ixy="0.01" ixz="0.01" iyy="0.01" iyz="0.01" izz="0.01" />
   </inertial>
@@ -78,5 +80,5 @@
     <origin xyz="0 0 0" rpy="0 0 -1.5707963" />
     <geometry>
-      <mesh filename="package://akros2_description/meshes/ld06.dae" />
+      <box size="0.038 0.0.0381 0.033"/>
     </geometry>
   </collision>
@@ -100,5 +102,5 @@
     <origin xyz="0 0 0" rpy="0 0 0" />
     <geometry>
-      <mesh filename="package://akros2_description/meshes/t265.dae" />
+      <box size="0.012 0.108 0.024"/>
     </geometry>
   </collision>
@@ -108,5 +110,5 @@
   <inertial>
     <origin xyz="0 0 0" rpy="0 0 0" />
-    <mass value="0.1" />
+    <mass value="0.055" />
     <inertia ixx="0.01" ixy="0.01" ixz="0.01" iyy="0.01" iyz="0.01" izz="0.01" />
   </inertial>
@@ -115,5 +117,5 @@
 <link name="wheel_lf">
   <inertial>
-    <mass value="0.1"/>
+    <mass value="0.075"/>
     <inertia ixx="5.1458e-5" iyy="5.1458e-5" izz="6.125e-5" ixy="0" ixz="0" iyz="0"/>
   </inertial>
@@ -128,5 +130,5 @@
     <origin xyz="0 0.01 0" rpy="1.5707963 0 0" />
     <geometry>
-      <cylinder length="0.035" radius="0.04"/>
+      <cylinder length="0.035" radius="0.038"/>
     </geometry>
   </collision>
@@ -135,5 +137,5 @@
 <link name="wheel_lb">
   <inertial>
-    <mass value="0.1"/>
+    <mass value="0.075"/>
     <inertia ixx="5.1458e-5" iyy="5.1458e-5" izz="6.125e-5" ixy="0" ixz="0" iyz="0"/>
   </inertial>
@@ -148,5 +150,5 @@
     <origin xyz="0 0.01 0" rpy="1.5707963 0 0" />
     <geometry>
-      <cylinder length="0.035" radius="0.04"/>
+      <cylinder length="0.035" radius="0.038"/>
     </geometry>
   </collision>
@@ -155,5 +157,5 @@
 <link name="wheel_rf">
   <inertial>
-    <mass value="0.1"/>
+    <mass value="0.075"/>
     <inertia ixx="5.1458e-5" iyy="5.1458e-5" izz="6.125e-5" ixy="0" ixz="0" iyz="0"/>
   </inertial>
@@ -168,5 +170,5 @@
     <origin xyz="0 -0.01 0" rpy="1.5707963 0 0" />
     <geometry>
-      <cylinder length="0.035" radius="0.04"/>
+      <cylinder length="0.035" radius="0.038"/>
     </geometry>
   </collision>
@@ -175,5 +177,5 @@
 <link name="wheel_rb">
   <inertial>
-    <mass value="0.1"/>
+    <mass value="0.075"/>
     <inertia ixx="5.1458e-5" iyy="5.1458e-5" izz="6.125e-5" ixy="0" ixz="0" iyz="0"/>
   </inertial>
@@ -188,5 +190,5 @@
     <origin xyz="0 -0.01 0" rpy="1.5707963 0 0" />
     <geometry>
-      <cylinder length="0.035" radius="0.04"/>
+      <cylinder length="0.035" radius="0.038"/>
     </geometry>
   </collision>

Commit message: updated collisions, moved to xacro, updated config for rviz and unity

File: urdf/akros2.urdf.xacro (robot description, xacro)
@@ -1,17 +1,13 @@
 <?xml version="1.0" encoding="utf-8"?>
-<robot name="akros" xmlns:xacro="http://ros.org/wiki/xacro">
-<!-- **** COLORS **** -->
-<material name="FlatBlack">
-    <color rgba="0.25 0.25 0.25 1"/>
-</material>
-<material name="DarkGrey">
-    <color rgba="0.5 0.5 0.5 1"/>
-</material>
-<material name="Grey">
-    <color rgba="0.75 0.75 0.75 1"/>
-</material>
-<material name="White">
-     <color rgba="1 1 1 1"/>
-</material>
+<robot name="akros2" xmlns:xacro="http://ros.org/wiki/xacro">
+<xacro:include filename="$(find akros2_description)/urdf/akros2.common.xacro"/>
+<xacro:include filename="$(find akros2_description)/urdf/akros2.control.xacro"/>
+<xacro:include filename="$(find akros2_description)/urdf/akros2.gazebo.xacro"/>
+<xacro:arg name="mesh_path" default="package://akros2_description/meshes/" />
+<xacro:arg name="unity" default="false" />
+<xacro:property name="mesh_path" value="$(arg mesh_path)" />
+<xacro:if value="$(arg unity)">
+  <xacro:property name="mesh_path" value="" />
+</xacro:if>
 <!-- **** LINKS **** -->
 <!-- BASE_LINK -->
@@ -20,13 +16,12 @@
     <origin xyz="0 0 0" rpy="0 0 0" />
     <geometry>
-      <mesh filename="package://akros2_description/meshes/base_module.dae" />
+      <mesh filename="${mesh_path}base_module.dae" />
     </geometry>
    <material name="White"/>
   </visual>
   <collision>
-    <origin xyz="0 0 0.0278" rpy="0 0 0" />
-    <geometry>
-      <box size="0.210 0.174 0.037"/>
-      <mesh filename="package://akros2_description/meshes/base_module.dae" />
+    <origin xyz="${base_offset_x} 0 ${base_height/2}" rpy="0 0 0" /> <!-- If needed: offset = 0.0278 -->
+    <geometry>
+      <box size="${base_length} ${base_width} ${base_height}"/>
     </geometry>
   </collision>
@@ -36,5 +31,5 @@
   <inertial>
     <origin xyz="0 0 0" rpy="0 0 0" />
-    <mass value="2.0"/>
+    <mass value="${base_mass}"/>
     <inertia ixx="0.015" iyy="0.0375" izz="0.0375" ixy="0" ixz="0" iyz="0"/>
   </inertial>
@@ -45,5 +40,5 @@
 <link name="nav_link">
   <inertial>
-    <mass value="0.5" />
+    <mass value="${nav_mass}" />
     <inertia ixx="0.01" ixy="0.01" ixz="0.01" iyy="0.01" iyz="0.01" izz="0.01" />
   </inertial>
@@ -51,13 +46,12 @@
     <origin xyz="0 0 -0.099" rpy="0 0 0" />
     <geometry>
-      <mesh filename="package://akros2_description/meshes/navigation_module.dae" />
-    </geometry>
-    <material name="DarkGrey"/>
-  </visual>
-  <collision>
-    <origin xyz="0 0 -0.099" rpy="0 0 0" />
-    <geometry>
-      <box size="0.2 0.154 0.037"/>
-      <mesh filename="package://akros2_description/meshes/navigation_module.dae" />
+      <mesh filename="${mesh_path}navigation_module.dae" />
+    </geometry>
+    <material name="DarkGrey"/>
+  </visual>
+  <collision>
+    <origin xyz="0 0 ${nav_height/2}" rpy="0 0 0" /> <!-- If needed: offset = -0.099 -->
+    <geometry>
+      <box size="${nav_length} ${nav_width} ${nav_height}"/>
     </geometry>
   </collision>
@@ -67,18 +61,18 @@
   <inertial>
     <origin xyz="0 0 0" rpy="0 0 0" />
-    <mass value="0.12" />
+    <mass value="${laser_mass}" />
     <inertia ixx="0.01" ixy="0.01" ixz="0.01" iyy="0.01" iyz="0.01" izz="0.01" />
   </inertial>
   <visual>
-    <origin xyz="0 0 0" rpy="0 0 -1.5707963" />
-    <geometry>
-      <mesh filename="package://akros2_description/meshes/ld06.dae" />
+    <origin xyz="0 0 0" rpy="0 0 ${minus_pi_by_two}" />
+    <geometry>
+      <mesh filename="${mesh_path}ld06.dae" />
     </geometry>
     <material name="FlatBlack"/>
   </visual>
   <collision>
-    <origin xyz="0 0 0" rpy="0 0 -1.5707963" />
-    <geometry>
-      <box size="0.038 0.0.0381 0.033"/>
+    <origin xyz="0 0 ${laser_height/2}" rpy="0 0 ${minus_pi_by_two}" />
+    <geometry>
+      <box size="${laser_length} ${laser_width} ${laser_height}"/>
     </geometry>
   </collision>
@@ -95,12 +89,12 @@
     <origin xyz="0 0 0" rpy="0 0 0" />
     <geometry>
-      <mesh filename="package://akros2_description/meshes/t265.dae" />
-    </geometry>
-    <material name="FlatBlack"/>
-  </visual>
-  <collision>
-    <origin xyz="0 0 0" rpy="0 0 0" />
-    <geometry>
-      <box size="0.012 0.108 0.024"/>
+      <mesh filename="${mesh_path}t265.dae" />
+    </geometry>
+    <material name="Grey"/>
+  </visual>
+  <collision>
+    <origin xyz="0 ${t265_offset_y} 0" rpy="0 0 0" />
+    <geometry>
+      <box size="${t265_length} ${t265_width} ${t265_height}"/>
     </geometry>
   </collision>
@@ -110,5 +104,5 @@
   <inertial>
     <origin xyz="0 0 0" rpy="0 0 0" />
-    <mass value="0.055" />
+    <mass value="${t265_mass}" />
     <inertia ixx="0.01" ixy="0.01" ixz="0.01" iyy="0.01" iyz="0.01" izz="0.01" />
   </inertial>
@@ -117,18 +111,18 @@
 <link name="wheel_lf">
   <inertial>
-    <mass value="0.075"/>
-    <inertia ixx="5.1458e-5" iyy="5.1458e-5" izz="6.125e-5" ixy="0" ixz="0" iyz="0"/>
-  </inertial>
-  <visual>
-    <origin xyz="0 0 0" rpy="0 0 0" />
-    <geometry>
-      <mesh filename="package://akros2_description/meshes/wheel_lf.dae" />
-    </geometry>
-    <material name="DarkGrey"/>
-  </visual>
-  <collision>
-    <origin xyz="0 0.01 0" rpy="1.5707963 0 0" />
-    <geometry>
-      <cylinder length="0.035" radius="0.038"/>
+    <mass value="${wheel_mass}"/>
+    <inertia ixx="5.1458e-5" iyy="5.1458e-5" izz="6.125e-5" ixy="0" ixz="0" iyz="0"/>
+  </inertial>
+  <visual>
+    <origin xyz="0 0 0" rpy="0 0 0" />
+    <geometry>
+      <mesh filename="${mesh_path}wheel_lf.dae" />
+    </geometry>
+    <material name="DarkGrey"/>
+  </visual>
+  <collision>
+    <origin xyz="0 ${wheel_height/2} 0" rpy="${pi_by_two} 0 0" /><!-- If needed: offset = 0.01 -->
+    <geometry>
+      <cylinder length="${wheel_height}" radius="${wheel_radius}"/>
     </geometry>
   </collision>
@@ -137,18 +131,18 @@
 <link name="wheel_lb">
   <inertial>
-    <mass value="0.075"/>
-    <inertia ixx="5.1458e-5" iyy="5.1458e-5" izz="6.125e-5" ixy="0" ixz="0" iyz="0"/>
-  </inertial>
-  <visual>
-    <origin xyz="0 0 0" rpy="0 0 0" />
-    <geometry>
-      <mesh filename="package://akros2_description/meshes/wheel_lb.dae" />
-    </geometry>
-    <material name="DarkGrey"/>
-  </visual>
-  <collision>
-    <origin xyz="0 0.01 0" rpy="1.5707963 0 0" />
-    <geometry>
-      <cylinder length="0.035" radius="0.038"/>
+    <mass value="${wheel_mass}"/>
+    <inertia ixx="5.1458e-5" iyy="5.1458e-5" izz="6.125e-5" ixy="0" ixz="0" iyz="0"/>
+  </inertial>
+  <visual>
+    <origin xyz="0 0 0" rpy="0 0 0" />
+    <geometry>
+      <mesh filename="${mesh_path}wheel_lb.dae" />
+    </geometry>
+    <material name="DarkGrey"/>
+  </visual>
+  <collision>
+    <origin xyz="0 ${wheel_height/2} 0" rpy="${pi_by_two} 0 0" /><!-- If needed: offset = 0.01 -->
+    <geometry>
+      <cylinder length="${wheel_height}" radius="${wheel_radius}"/>
     </geometry>
   </collision>
@@ -157,18 +151,18 @@
 <link name="wheel_rf">
   <inertial>
-    <mass value="0.075"/>
-    <inertia ixx="5.1458e-5" iyy="5.1458e-5" izz="6.125e-5" ixy="0" ixz="0" iyz="0"/>
-  </inertial>
-  <visual>
-    <origin xyz="0 0 0" rpy="0 0 0" />
-    <geometry>
-      <mesh filename="package://akros2_description/meshes/wheel_rf.dae" />
-    </geometry>
-    <material name="DarkGrey"/>
-  </visual>
-  <collision>
-    <origin xyz="0 -0.01 0" rpy="1.5707963 0 0" />
-    <geometry>
-      <cylinder length="0.035" radius="0.038"/>
+    <mass value="${wheel_mass}"/>
+    <inertia ixx="5.1458e-5" iyy="5.1458e-5" izz="6.125e-5" ixy="0" ixz="0" iyz="0"/>
+  </inertial>
+  <visual>
+    <origin xyz="0 0 0" rpy="0 0 0" />
+    <geometry>
+      <mesh filename="${mesh_path}wheel_rf.dae" />
+    </geometry>
+    <material name="DarkGrey"/>
+  </visual>
+  <collision>
+    <origin xyz="0 ${-1*(wheel_height/2)} 0" rpy="${pi_by_two} 0 0" /><!-- If needed: offset = 0.01 -->
+    <geometry>
+      <cylinder length="${wheel_height}" radius="${wheel_radius}"/>
     </geometry>
   </collision>
@@ -177,18 +171,18 @@
 <link name="wheel_rb">
   <inertial>
-    <mass value="0.075"/>
-    <inertia ixx="5.1458e-5" iyy="5.1458e-5" izz="6.125e-5" ixy="0" ixz="0" iyz="0"/>
-  </inertial>
-  <visual>
-    <origin xyz="0 0 0" rpy="0 0 0" />
-    <geometry>
-      <mesh filename="package://akros2_description/meshes/wheel_rb.dae" />
-    </geometry>
-    <material name="DarkGrey"/>
-  </visual>
-  <collision>
-    <origin xyz="0 -0.01 0" rpy="1.5707963 0 0" />
-    <geometry>
-      <cylinder length="0.035" radius="0.038"/>
+    <mass value="${wheel_mass}"/>
+    <inertia ixx="5.1458e-5" iyy="5.1458e-5" izz="6.125e-5" ixy="0" ixz="0" iyz="0"/>
+  </inertial>
+  <visual>
+    <origin xyz="0 0 0" rpy="0 0 0" />
+    <geometry>
+      <mesh filename="${mesh_path}wheel_rb.dae" />
+    </geometry>
+    <material name="DarkGrey"/>
+  </visual>
+  <collision>
+    <origin xyz="0 ${-1*(wheel_height/2)} 0" rpy="${pi_by_two} 0 0" /><!-- If needed: offset = 0.01 -->
+    <geometry>
+      <cylinder length="${wheel_height}" radius="${wheel_radius}"/>
     </geometry>
   </collision>
@@ -199,5 +193,5 @@
   <parent link="t265_pose_frame"/>
   <child link="base_link"/>
-  <origin xyz="-0.094 0 -0.115"/>
+  <origin xyz="${pose_base_offset_x} 0 ${pose_base_offset_z}"/>
 </joint>
 <!-- T265_POSE_INERTIAL TO T265_POSE_FRAME -->
@@ -223,5 +217,5 @@
   <parent link="base_link"/>
   <child link="nav_link"/>
-  <origin xyz="0 0 0.099"/>
+  <origin xyz="0 0 ${base_height}"/>
   <axis xyz="0 0 0"/>
 </joint>
@@ -230,5 +224,5 @@
   <parent link="nav_link"/>
   <child link="laser_link"/>
-  <origin xyz="0.0632 0 0.0155"/>
+  <origin xyz="${nav_laser_offset_x} 0 ${nav_height/2}"/>
 </joint>
 <!-- LASER_FRAME TO LASER_LINK -->
@@ -236,5 +230,5 @@
   <parent link="laser_link"/>
   <child link="laser_frame"/>
-  <origin xyz="0 0 0.0255"/>
+  <origin xyz="0 0 ${laser_frame_offset_z}"/>
 </joint>
 <!-- IMU_LINK TO BASE_LINK -->
@@ -254,136 +248,27 @@
   <parent link="base_link" />
   <child link="wheel_lf" />
-  <origin xyz="0.0495 0.078 0.021" rpy="0 0 0" />
-  <axis xyz="0 1 0" />
-</joint>
-<transmission name="trans_lf">
-  <type>transmission_interface/SimpleTransmission</type>
-  <joint name="joint_lf">
-    <hardwareInterface>hardware_interface/VelocityJointInterface</hardwareInterface>
-  </joint>
-  <actuator name="motor_lf">
-    <hardwareInterface>hardware_interface/VelocityJointInterface</hardwareInterface>
-    <mechanicalReduction>1</mechanicalReduction>
-  </actuator>
-</transmission>
+  <origin xyz="${joint_offset_x} ${joint_offset_y} ${joint_offset_z}" rpy="0 0 0" />
+  <axis xyz="0 1 0" />
+</joint>
 <!-- WHEEL_LB TO BASE_LINK -->
 <joint name="joint_lb" type="continuous">
   <parent link="base_link" />
   <child link="wheel_lb" />
-  <origin xyz="-0.0495 0.077 0.021" rpy="0 0 0" />
-  <axis xyz="0 1 0" />
-</joint>
-<transmission name="trans_lb">
-  <type>transmission_interface/SimpleTransmission</type>
-  <joint name="joint_lb">
-    <hardwareInterface>hardware_interface/VelocityJointInterface</hardwareInterface>
-  </joint>
-  <actuator name="motor_lb">
-    <hardwareInterface>hardware_interface/VelocityJointInterface</hardwareInterface>
-    <mechanicalReduction>1</mechanicalReduction>
-  </actuator>
-</transmission>
+  <origin xyz="${-1*joint_offset_x} ${joint_offset_y} ${joint_offset_z}" rpy="0 0 0" />
+  <axis xyz="0 1 0" />
+</joint>
 <!-- WHEEL_RF TO BASE_LINK -->
 <joint name="joint_rf" type="continuous">
   <parent link="base_link" />
   <child link="wheel_rf" />
-  <origin xyz="0.0495 -0.078 0.021" rpy="0 0 0" />
-  <axis xyz="0 1 0" />
-</joint>
-<transmission name="trans_rf">
-  <type>transmission_interface/SimpleTransmission</type>
-  <joint name="joint_rf">
-    <hardwareInterface>hardware_interface/VelocityJointInterface</hardwareInterface>
-  </joint>
-  <actuator name="motor_rf">
-    <hardwareInterface>hardware_interface/VelocityJointInterface</hardwareInterface>
-    <mechanicalReduction>1</mechanicalReduction>
-  </actuator>
-</transmission>
+  <origin xyz="${joint_offset_x} ${-1*joint_offset_y} ${joint_offset_z}" rpy="0 0 0" />
+  <axis xyz="0 1 0" />
+</joint>
 <!-- WHEEL_RB TO BASE_LINK -->
 <joint name="joint_rb" type="continuous">
   <parent link="base_link" />
   <child link="wheel_rb" />
-  <origin xyz="-0.0495 -0.078 0.021" rpy="0 0 0" />
-  <axis xyz="0 1 0" />
-</joint>
-<transmission name="trans_rb">
-  <type>transmission_interface/SimpleTransmission</type>
-  <joint name="joint_rb">
-    <hardwareInterface>hardware_interface/VelocityJointInterface</hardwareInterface>
-  </joint>
-  <actuator name="motor_rb">
-    <hardwareInterface>hardware_interface/VelocityJointInterface</hardwareInterface>
-    <mechanicalReduction>1</mechanicalReduction>
-  </actuator>
-</transmission>
-<!-- **** GAZEBO **** -->
-<gazebo reference="base_link">
-  <material>Gazebo/White</material>
-</gazebo>
-<gazebo reference="nav_link">
-  <material>Gazebo/DarkGrey</material>
-</gazebo>
-<gazebo reference="laser_link">
-  <material>Gazebo/FlatBlack</material>
-</gazebo>
-<gazebo reference="t265_pose_frame">
-  <material>Gazebo/FlatBlack</material>
-</gazebo>
-<gazebo reference="wheel_lf">
-  <material>Gazebo/DarkGrey</material>
-</gazebo>
-<gazebo reference="wheel_lb">
-  <material>Gazebo/DarkGrey</material>
-</gazebo>
-<gazebo reference="wheel_rf">
-  <material>Gazebo/DarkGrey</material>
-</gazebo>
-<gazebo reference="wheel_rb">
-  <material>Gazebo/DarkGrey</material>
-</gazebo>
-<gazebo reference="laser_frame">
-  <sensor type="ray" name="head_ld06_sensor">
-    <pose>0 0 0.06 0 0 0</pose>
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
Commit message: updated xacro

File: urdf/akros2.urdf.xacro (robot description, xacro)
@@ -4,5 +4,5 @@
 <xacro:include filename="$(find akros2_description)/urdf/akros2.control.xacro"/>
 <xacro:include filename="$(find akros2_description)/urdf/akros2.gazebo.xacro"/>
-<xacro:arg name="mesh_path" default="package://akros2_description/meshes/" />
+<xacro:arg name="mesh_path" default="package://akros2_description/meshes/" /> <!-- HTTPS URL also works here -->
 <xacro:arg name="unity" default="false" />
 <xacro:property name="mesh_path" value="$(arg mesh_path)" />
@@ -119,5 +119,5 @@
       <mesh filename="${mesh_path}wheel_lf.dae" />
     </geometry>
-    <material name="DarkGrey"/>
+    <material name="FlatBlack"/>
   </visual>
   <collision>
@@ -139,5 +139,5 @@
       <mesh filename="${mesh_path}wheel_lb.dae" />
     </geometry>
-    <material name="DarkGrey"/>
+    <material name="FlatBlack"/>
   </visual>
   <collision>
@@ -159,5 +159,5 @@
       <mesh filename="${mesh_path}wheel_rf.dae" />
     </geometry>
-    <material name="DarkGrey"/>
+    <material name="FlatBlack"/>
   </visual>
   <collision>
@@ -179,5 +179,5 @@
       <mesh filename="${mesh_path}wheel_rb.dae" />
     </geometry>
-    <material name="DarkGrey"/>
+    <material name="FlatBlack"/>
   </visual>
   <collision>
