Commit message: updated inertia values according to geometry size

File: urdf/akros2.common.xacro (robot description, xacro)
@@ -31,4 +31,19 @@
 <xacro:property name="joint_offset_y" value="0.078" />
 <xacro:property name="joint_offset_z" value="0.021" />
+<xacro:macro name="cylinder_inertia" params="m r h">
+  <inertia  ixx="${m*(3*r*r+h*h)/12}" ixy = "0" ixz = "0"
+            iyy="${m*(3*r*r+h*h)/12}" iyz = "0"
+            izz="${m*r*r/2}" />
+</xacro:macro>
+<xacro:macro name="box_inertia" params="m x y z">
+  <inertia  ixx="${m*(y*y+z*z)/12}" ixy = "0" ixz = "0"
+            iyy="${m*(x*x+z*z)/12}" iyz = "0"
+            izz="${m*(x*x+z*z)/12}" />
+</xacro:macro>
+<xacro:macro name="sphere_inertia" params="m r">
+  <inertia  ixx="${2*m*r*r/5}" ixy = "0" ixz = "0"
+            iyy="${2*m*r*r/5}" iyz = "0"
+            izz="${2*m*r*r/5}" />
+</xacro:macro>
 <material name="FlatBlack">
     <color rgba="0.25 0.25 0.25 1"/>

File: urdf/akros2.urdf (robot description, URDF)
Before this commit: robot akros2, 14 links, 13 joints
Links:
- link base_link: geometry collision box size=0.21 0.154 0.099; visual mesh filename=package://akros2_description/meshes/base_module.dae
- link laser_link: geometry collision box size=0.038 0.0381 0.033; visual mesh filename=package://akros2_description/meshes/ld06.dae
- link nav_link: geometry collision box size=0.2 0.154 0.031; visual mesh filename=package://akros2_description/meshes/navigation_module.dae
- link t265_pose_frame: geometry collision box size=0.012 0.108 0.024; visual mesh filename=package://akros2_description/meshes/t265.dae
- link wheel_lb: geometry collision cylinder length=0.034 radius=0.038; visual mesh filename=package://akros2_description/meshes/wheel_lb.dae
- link wheel_lf: geometry collision cylinder length=0.034 radius=0.038; visual mesh filename=package://akros2_description/meshes/wheel_lf.dae
- link wheel_rb: geometry collision cylinder length=0.034 radius=0.038; visual mesh filename=package://akros2_description/meshes/wheel_rb.dae
- link wheel_rf: geometry collision cylinder length=0.034 radius=0.038; visual mesh filename=package://akros2_description/meshes/wheel_rf.dae

File: urdf/akros2.urdf.xacro (robot description, xacro)
@@ -21,5 +21,5 @@
   </visual>
   <collision>
-    <origin xyz="${base_offset_x} 0 ${base_height/2}" rpy="0 0 0" /> <!-- If needed: offset = 0.0278 -->
+    <origin xyz="${base_offset_x} 0 ${base_height/2}" rpy="0 0 0" /> <!-- If needed: offset from ground = 0.0278 -->
     <geometry>
       <box size="${base_length} ${base_width} ${base_height}"/>
@@ -32,5 +32,5 @@
     <origin xyz="0 0 0" rpy="0 0 0" />
     <mass value="${base_mass}"/>
-    <inertia ixx="0.015" iyy="0.0375" izz="0.0375" ixy="0" ixz="0" iyz="0"/>
+    <xacro:box_inertia m="${base_mass}" x="${base_length}" y="${base_width}" z="${base_height}"/>
   </inertial>
 </link>
@@ -41,5 +41,5 @@
   <inertial>
     <mass value="${nav_mass}" />
-    <inertia ixx="0.01" ixy="0.01" ixz="0.01" iyy="0.01" iyz="0.01" izz="0.01" />
+    <xacro:box_inertia m="${nav_mass}" x="${nav_length}" y="${nav_width}" z="${nav_height}"/>
   </inertial>
   <visual>
@@ -51,5 +51,5 @@
   </visual>
   <collision>
-    <origin xyz="0 0 ${nav_height/2}" rpy="0 0 0" /> <!-- If needed: offset = -0.099 -->
+    <origin xyz="0 0 ${nav_height/2}" rpy="0 0 0" /> <!-- If needed: offset from base_link = -0.099 -->
     <geometry>
       <box size="${nav_length} ${nav_width} ${nav_height}"/>
@@ -62,5 +62,5 @@
     <origin xyz="0 0 0" rpy="0 0 0" />
     <mass value="${laser_mass}" />
-    <inertia ixx="0.01" ixy="0.01" ixz="0.01" iyy="0.01" iyz="0.01" izz="0.01" />
+    <xacro:box_inertia m="${laser_mass}" x="${laser_length}" y="${laser_width}" z="${laser_height}"/>
   </inertial>
   <visual>
@@ -105,5 +105,5 @@
     <origin xyz="0 0 0" rpy="0 0 0" />
     <mass value="${t265_mass}" />
-    <inertia ixx="0.01" ixy="0.01" ixz="0.01" iyy="0.01" iyz="0.01" izz="0.01" />
+    <xacro:box_inertia m="${t265_mass}" x="${t265_length}" y="${t265_width}" z="${t265_height}"/>
   </inertial>
 </link>
@@ -112,5 +112,5 @@
   <inertial>
     <mass value="${wheel_mass}"/>
-    <inertia ixx="5.1458e-5" iyy="5.1458e-5" izz="6.125e-5" ixy="0" ixz="0" iyz="0"/>
+    <xacro:cylinder_inertia m="${wheel_mass}" r="${wheel_radius}" h="${wheel_height}"/>
   </inertial>
   <visual>
@@ -122,5 +122,5 @@
   </visual>
   <collision>
-    <origin xyz="0 ${wheel_height/2} 0" rpy="${pi_by_two} 0 0" /><!-- If needed: offset = 0.01 -->
+    <origin xyz="0 ${wheel_height/2} 0" rpy="${pi_by_two} 0 0" /><!-- If needed: offset from joint = 0.01 -->
     <geometry>
       <cylinder length="${wheel_height}" radius="${wheel_radius}"/>
@@ -132,5 +132,5 @@
   <inertial>
     <mass value="${wheel_mass}"/>
-    <inertia ixx="5.1458e-5" iyy="5.1458e-5" izz="6.125e-5" ixy="0" ixz="0" iyz="0"/>
+    <xacro:cylinder_inertia m="${wheel_mass}" r="${wheel_radius}" h="${wheel_height}"/>
   </inertial>
   <visual>
@@ -142,5 +142,5 @@
   </visual>
   <collision>
-    <origin xyz="0 ${wheel_height/2} 0" rpy="${pi_by_two} 0 0" /><!-- If needed: offset = 0.01 -->
+    <origin xyz="0 ${wheel_height/2} 0" rpy="${pi_by_two} 0 0" /><!-- If needed: offset from joint = 0.01 -->
     <geometry>
       <cylinder length="${wheel_height}" radius="${wheel_radius}"/>
@@ -152,5 +152,5 @@
   <inertial>
     <mass value="${wheel_mass}"/>
-    <inertia ixx="5.1458e-5" iyy="5.1458e-5" izz="6.125e-5" ixy="0" ixz="0" iyz="0"/>
+    <xacro:cylinder_inertia m="${wheel_mass}" r="${wheel_radius}" h="${wheel_height}"/>
   </inertial>
   <visual>
@@ -162,5 +162,5 @@
   </visual>
   <collision>
-    <origin xyz="0 ${-1*(wheel_height/2)} 0" rpy="${pi_by_two} 0 0" /><!-- If needed: offset = 0.01 -->
+    <origin xyz="0 ${-1*(wheel_height/2)} 0" rpy="${pi_by_two} 0 0" /><!-- If needed: offset from joint = 0.01 -->
     <geometry>
       <cylinder length="${wheel_height}" radius="${wheel_radius}"/>
@@ -172,5 +172,5 @@
   <inertial>
     <mass value="${wheel_mass}"/>
-    <inertia ixx="5.1458e-5" iyy="5.1458e-5" izz="6.125e-5" ixy="0" ixz="0" iyz="0"/>
+    <xacro:cylinder_inertia m="${wheel_mass}" r="${wheel_radius}" h="${wheel_height}"/>
   </inertial>
   <visual>
@@ -182,5 +182,5 @@
   </visual>
   <collision>
-    <origin xyz="0 ${-1*(wheel_height/2)} 0" rpy="${pi_by_two} 0 0" /><!-- If needed: offset = 0.01 -->
+    <origin xyz="0 ${-1*(wheel_height/2)} 0" rpy="${pi_by_two} 0 0" /><!-- If needed: offset from joint = 0.01 -->
     <geometry>
       <cylinder length="${wheel_height}" radius="${wheel_radius}"/>
