Commit message: add files for akros2_omni

File: urdf/akros2/akros2.urdf (robot description, URDF)
Before this commit: robot akros2, 14 links, 13 joints
Links:
- link base_link: geometry collision box size=0.21 0.154 0.099; visual mesh filename=package://akros2_description/meshes/akros2/base_module.dae
- link laser_link: geometry collision box size=0.038 0.0381 0.033; visual mesh filename=package://akros2_description/meshes/akros2/ld06.dae
- link nav_link: geometry collision box size=0.2 0.154 0.031; visual mesh filename=package://akros2_description/meshes/akros2/navigation_modul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
- link t265_pose_frame: geometry collision box size=0.012 0.108 0.024; visual mesh filename=package://akros2_description/meshes/akros2/t265.dae
- link wheel_lb: geometry collision cylinder length=0.034 radius=0.038; visual mesh filename=package://akros2_description/meshes/akros2/wheel_lb.dae
- link wheel_lf: geometry collision cylinder length=0.034 radius=0.038; visual mesh filename=package://akros2_description/meshes/akros2/wheel_lf.dae
- link wheel_rb: geometry collision cylinder length=0.034 radius=0.038; visual mesh filename=package://akros2_description/meshes/akros2/wheel_rb.dae
- link wheel_rf: geometry collision cylinder length=0.034 radius=0.038; visual mesh filename=package://akros2_description/meshes/akros2/wheel_rf.dae

File: urdf/akros2_omni/akros2_omni.urdf.xacro (robot description, xacro)
@@ -1,8 +1,8 @@
 <?xml version="1.0" encoding="utf-8"?>
 <robot name="akros2" xmlns:xacro="http://ros.org/wiki/xacro">
-<xacro:include filename="$(find akros2_description)/urdf/akros2.common.xacro"/>
-<xacro:include filename="$(find akros2_description)/urdf/akros2.control.xacro"/>
-<xacro:include filename="$(find akros2_description)/urdf/akros2.gazebo.xacro"/>
-<xacro:arg name="mesh_path" default="package://akros2_description/meshes/" /> <!-- HTTPS URL also works here -->
+<xacro:include filename="$(find akros2_description)/urdf/akros2_omni/akros2_omni.common.xacro"/>
+<xacro:include filename="$(find akros2_description)/urdf/akros2_omni/akros2_omni.control.xacro"/>
+<xacro:include filename="$(find akros2_description)/urdf/akros2_omni/akros2_omni.gazebo.xacro"/>
+<xacro:arg name="mesh_path" default="package://akros2_description/meshes/akros2_omni/" /> <!-- HTTPS URL also works here -->
 <xacro:arg name="unity" default="false" />
 <xacro:property name="mesh_path" value="$(arg mesh_path)" />
@@ -84,30 +84,6 @@
 <!-- IMU_FRAME -->
 <link name="imu_frame"/>
-<!-- T265 TRACKING CAMERA (T265_POSE_FRAME AS WORKAROUND TO KEEP TREE CONTINUOUS)-->
-<link name="t265_pose_frame">
-  <visual>
-    <origin xyz="0 0 0" rpy="0 0 0" />
-    <geometry>
-      <mesh filename="${mesh_path}t265.dae" />
-    </geometry>
-    <material name="Grey"/>
-  </visual>
-  <collision>
-    <origin xyz="0 ${t265_offset_y} 0" rpy="0 0 0" />
-    <geometry>
-      <box size="${t265_length} ${t265_width} ${t265_height}"/>
-    </geometry>
-  </collision>
-</link>
-<!-- T265 TRACKING CAMERA (T265_POSE_INERTIAL)-->
-<link name="t265_pose_inertial">
-  <inertial>
-    <origin xyz="0 0 0" rpy="0 0 0" />
-    <mass value="${t265_mass}" />
-    <xacro:box_inertia m="${t265_mass}" x="${t265_length}" y="${t265_width}" z="${t265_height}"/>
-  </inertial>
-</link>
-<!-- WHEEL LEFT FRONT -->
-<link name="wheel_lf">
+<!-- WHEEL FRONT -->
+<link name="wheel_f">
   <inertial>
     <mass value="${wheel_mass}"/>
@@ -117,5 +93,5 @@
     <origin xyz="0 0 0" rpy="0 0 0" />
     <geometry>
-      <mesh filename="${mesh_path}wheel_lf.dae" />
+      <mesh filename="${mesh_path}wheel_f.dae" />
     </geometry>
     <material name="FlatBlack"/>
@@ -128,6 +104,6 @@
   </collision>
 </link>
-<!-- WHEEL LEFT BACK -->
-<link name="wheel_lb">
+<!-- WHEEL LEFT (BACK) -->
+<link name="wheel_l">
   <inertial>
     <mass value="${wheel_mass}"/>
@@ -137,5 +113,5 @@
     <origin xyz="0 0 0" rpy="0 0 0" />
     <geometry>
-      <mesh filename="${mesh_path}wheel_lb.dae" />
+      <mesh filename="${mesh_path}wheel_l.dae" />
     </geometry>
     <material name="FlatBlack"/>
@@ -148,6 +124,6 @@
   </collision>
 </link>
-<!-- WHEEL RIGHT FRONT -->
-<link name="wheel_rf">
+<!-- WHEEL RIGHT (BACK) -->
+<link name="wheel_r">
   <inertial>
     <mass value="${wheel_mass}"/>
@@ -157,5 +133,5 @@
     <origin xyz="0 0 0" rpy="0 0 0" />
     <geometry>
-      <mesh filename="${mesh_path}wheel_rf.dae" />
+      <mesh filename="${mesh_path}wheel_r.dae" />
     </geometry>
     <material name="FlatBlack"/>
@@ -168,37 +144,5 @@
   </collision>
 </link>
-<!-- WHEEL RIGHT BACK -->
-<link name="wheel_rb">
-  <inertial>
-    <mass value="${wheel_mass}"/>
-    <xacro:cylinder_inertia m="${wheel_mass}" r="${wheel_radius}" h="${wheel_height}"/>
-  </inertial>
-  <visual>
-    <origin xyz="0 0 0" rpy="0 0 0" />
-    <geometry>
-      <mesh filename="${mesh_path}wheel_rb.dae" />
-    </geometry>
-    <material name="FlatBlack"/>
-  </visual>
-  <collision>
-    <origin xyz="0 ${-1*(wheel_height/2)} 0" rpy="${pi_by_two} 0 0" /><!-- If needed: offset from joint = 0.01 -->
-    <geometry>
-      <cylinder length="${wheel_height}" radius="${wheel_radius}"/>
-    </geometry>
-  </collision>
-</link>
 <!-- **** JOINTS **** -->
-<!-- BASE_LINK TO T265_POSE_FRAME -->
-<joint name="pose_base_fixed" type="fixed">
-  <parent link="t265_pose_frame"/>
-  <child link="base_link"/>
-  <origin xyz="${pose_base_offset_x} 0 ${pose_base_offset_z}"/>
-</joint>
-<!-- T265_POSE_INERTIAL TO T265_POSE_FRAME -->
-<joint name="pose_inertial_fixed" type="fixed">
-  <parent link="t265_pose_frame"/>
-  <child link="t265_pose_inertial"/>
-  <origin xyz="0 0 0"/>
-</joint>
 <!-- BASE_LINK_INERTIAL TO BASE_LINK -->
 <joint name="base_inertial_fixed" type="fixed">
@@ -244,31 +188,24 @@
   <origin xyz="0 0 0"/>
 </joint>
-<!-- WHEEL_LF TO BASE_LINK -->
-<joint name="joint_lf" type="continuous">
+<!-- WHEEL_F TO BASE_LINK -->
+<joint name="joint_f" type="continuous">
   <parent link="base_link" />
-  <child link="wheel_lf" />
+  <child link="wheel_f" />
   <origin xyz="${joint_offset_x} ${joint_offset_y} ${joint_offset_z}" rpy="0 0 0" />
   <axis xyz="0 1 0" />
 </joint>
-<!-- WHEEL_LB TO BASE_LINK -->
-<joint name="joint_lb" type="continuous">
+<!-- WHEEL_L TO BASE_LINK -->
+<joint name="joint_l" type="continuous">
   <parent link="base_link" />
-  <child link="wheel_lb" />
+  <child link="wheel_l" />
   <origin xyz="${-1*joint_offset_x} ${joint_offset_y} ${joint_offset_z}" rpy="0 0 0" />
   <axis xyz="0 1 0" />
 </joint>
-<!-- WHEEL_RF TO BASE_LINK -->
-<joint name="joint_rf" type="continuous">
+<!-- WHEEL_R TO BASE_LINK -->
+<joint name="joint_r" type="continuous">
   <parent link="base_link" />
-  <child link="wheel_rf" />
+  <child link="wheel_r" />
   <origin xyz="${joint_offset_x} ${-1*joint_offset_y} ${joint_offset_z}" rpy="0 0 0" />
   <axis xyz="0 1 0" />
 </joint>
-<!-- WHEEL_RB TO BASE_LINK -->
-<joint name="joint_rb" type="continuous">
-  <parent link="base_link" />
-  <child link="wheel_rb" />
-  <origin xyz="${-1*joint_offset_x} ${-1*joint_offset_y} ${joint_offset_z}" rpy="0 0 0" />
-  <axis xyz="0 1 0" />
-</joint>
 </robot>
