Commit message: Update akros2_mecanum.urdf.xacro

File: urdf/akros2_mecanum/akros2_mecanum.urdf.xacro (robot description, xacro)
@@ -88,5 +88,5 @@
   <inertial>
     <mass value="${wheel_mass}"/>
-    <xacro:cylinder_inertia m="${wheel_mass}" r="${wheel_radius}" h="${wheel_height}"/>
+    <xacro:cylinder_inertia m="${wheel_mass}" r="${wheel_radius}" h="${wheel_thickness}"/>
   </inertial>
   <visual>
@@ -98,7 +98,7 @@
   </visual>
   <collision>
-    <origin xyz="0 ${wheel_height/2} 0" rpy="${pi_by_two} 0 0" />
-    <geometry>
-      <cylinder length="${wheel_height}" radius="${wheel_radius}"/>
+    <origin xyz="0 ${wheel_thickness/2} 0" rpy="${pi_by_two} 0 0" />
+    <geometry>
+      <cylinder length="${wheel_thickness}" radius="${wheel_radius}"/>
     </geometry>
   </collision>
@@ -108,5 +108,5 @@
   <inertial>
     <mass value="${wheel_mass}"/>
-    <xacro:cylinder_inertia m="${wheel_mass}" r="${wheel_radius}" h="${wheel_height}"/>
+    <xacro:cylinder_inertia m="${wheel_mass}" r="${wheel_radius}" h="${wheel_thickness}"/>
   </inertial>
   <visual>
@@ -118,7 +118,7 @@
   </visual>
   <collision>
-    <origin xyz="0 ${wheel_height/2} 0" rpy="${pi_by_two} 0 0" />
-    <geometry>
-      <cylinder length="${wheel_height}" radius="${wheel_radius}"/>
+    <origin xyz="0 ${wheel_thickness/2} 0" rpy="${pi_by_two} 0 0" />
+    <geometry>
+      <cylinder length="${wheel_thickness}" radius="${wheel_radius}"/>
     </geometry>
   </collision>
@@ -128,5 +128,5 @@
   <inertial>
     <mass value="${wheel_mass}"/>
-    <xacro:cylinder_inertia m="${wheel_mass}" r="${wheel_radius}" h="${wheel_height}"/>
+    <xacro:cylinder_inertia m="${wheel_mass}" r="${wheel_radius}" h="${wheel_thickness}"/>
   </inertial>
   <visual>
@@ -138,7 +138,7 @@
   </visual>
   <collision>
-    <origin xyz="0 ${-1*(wheel_height/2)} 0" rpy="${pi_by_two} 0 0" />
-    <geometry>
-      <cylinder length="${wheel_height}" radius="${wheel_radius}"/>
+    <origin xyz="0 ${-1*(wheel_thickness/2)} 0" rpy="${pi_by_two} 0 0" />
+    <geometry>
+      <cylinder length="${wheel_thickness}" radius="${wheel_radius}"/>
     </geometry>
   </collision>
@@ -148,5 +148,5 @@
   <inertial>
     <mass value="${wheel_mass}"/>
-    <xacro:cylinder_inertia m="${wheel_mass}" r="${wheel_radius}" h="${wheel_height}"/>
+    <xacro:cylinder_inertia m="${wheel_mass}" r="${wheel_radius}" h="${wheel_thickness}"/>
   </inertial>
   <visual>
@@ -158,7 +158,7 @@
   </visual>
   <collision>
-    <origin xyz="0 ${-1*(wheel_height/2)} 0" rpy="${pi_by_two} 0 0" />
-    <geometry>
-      <cylinder length="${wheel_height}" radius="${wheel_radius}"/>
+    <origin xyz="0 ${-1*(wheel_thickness/2)} 0" rpy="${pi_by_two} 0 0" />
+    <geometry>
+      <cylinder length="${wheel_thickness}" radius="${wheel_radius}"/>
     </geometry>
   </collision>
