Commit message: divide into akros2_mecanum, akros2_omni, update readme

File: urdf/akros2_mecanum/akros2_mecanum.common.xacro (robot description, xacro)
@@ -1,4 +1,4 @@
 <?xml version="1.0" encoding="utf-8"?>
-<robot name="akros2_common" xmlns:xacro="http://ros.org/wiki/xacro">
+<robot name="mecanum_common" xmlns:xacro="http://ros.org/wiki/xacro">
 <xacro:property name="pi_by_two" value="1.5707963" />
 <xacro:property name="minus_pi_by_two" value="-1.5707963" />
@@ -16,14 +16,7 @@
 <xacro:property name="laser_width" value="0.0381" />
 <xacro:property name="laser_height" value="0.033" />
-<xacro:property name="t265_mass" value="0.055" />
-<xacro:property name="t265_length" value="0.012" />
-<xacro:property name="t265_width" value="0.108" />
-<xacro:property name="t265_height" value="0.024" />
-<xacro:property name="t265_offset_y" value="0.00125" />
 <xacro:property name="wheel_radius" value="0.038" />
 <xacro:property name="wheel_mass" value="0.075" />
 <xacro:property name="wheel_height" value="0.034" />
-<xacro:property name="pose_base_offset_x" value="-0.094" />
-<xacro:property name="pose_base_offset_z" value="-0.115" />
 <xacro:property name="nav_laser_offset_x" value="0.0632" />
 <xacro:property name="laser_frame_offset_z" value="0.0255" />

File: urdf/akros2_mecanum/akros2_mecanum.control.xacro (robot description, xacro)
@@ -1,4 +1,4 @@
 <?xml version="1.0" encoding="utf-8"?>
-<robot name="akros2_control" xmlns:xacro="http://ros.org/wiki/xacro">
+<robot name="mecanum_control" xmlns:xacro="http://ros.org/wiki/xacro">
 <!-- WHEEL_LF TRANSMISSION -->
 <transmission name="trans_lf">

File: urdf/akros2_mecanum/akros2_mecanum.gazebo.xacro (robot description, xacro)
@@ -1,4 +1,4 @@
 <?xml version="1.0" encoding="utf-8"?>
-<robot name="akros2_gazebo" xmlns:xacro="http://ros.org/wiki/xacro">
+<robot name="mecanum_gazebo" xmlns:xacro="http://ros.org/wiki/xacro">
 <gazebo reference="base_link">
   <material>Gazebo/White</material>
@@ -9,7 +9,4 @@
 <gazebo reference="laser_link">
   <material>Gazebo/FlatBlack</material>
-</gazebo>
-<gazebo reference="t265_pose_frame">
-  <material>Gazebo/Grey</material>
 </gazebo>
 <gazebo reference="wheel_lf">

File: urdf/akros2_mecanum/akros2_mecanum.urdf (robot description, URDF)
Before this commit: robot akros2, 14 links, 13 joints
Links:
- removed link t265_pose_frame
- removed link t265_pose_inertial
- link base_link: geometry collision box size=0.21 0.154 0.099; visual mesh filename=package://akros2_description/meshes/akros2_mecanum/base_mod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
- link laser_link: geometry collision box size=0.038 0.0381 0.033; visual mesh filename=package://akros2_description/meshes/akros2_mecanum/ld06.dae
- link nav_link: geometry collision box size=0.2 0.154 0.031; visual mesh filename=package://akros2_description/meshes/akros2_mecanum/navigati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
- link wheel_lb: geometry collision cylinder length=0.034 radius=0.038; visual mesh filename=package://akros2_description/meshes/akros2_mecanum/wheel_lb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
- link wheel_lf: geometry collision cylinder length=0.034 radius=0.038; visual mesh filename=package://akros2_description/meshes/akros2_mecanum/wheel_lf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
- link wheel_rb: geometry collision cylinder length=0.034 radius=0.038; visual mesh filename=package://akros2_description/meshes/akros2_mecanum/wheel_rb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
- link wheel_rf: geometry collision cylinder length=0.034 radius=0.038; visual mesh filename=package://akros2_description/meshes/akros2_mecanum/wheel_rf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
Joints:
- removed joint pose_base_fixed
- removed joint pose_inertial_fixed

File: urdf/akros2_mecanum/akros2_mecanum.urdf.xacro (robot description, xacro)
@@ -1,8 +1,8 @@
 <?xml version="1.0" encoding="utf-8"?>
-<robot name="akros2" xmlns:xacro="http://ros.org/wiki/xacro">
-<xacro:include filename="$(find akros2_description)/urdf/akros2/akros2.common.xacro"/>
-<xacro:include filename="$(find akros2_description)/urdf/akros2/akros2.control.xacro"/>
-<xacro:include filename="$(find akros2_description)/urdf/akros2/akros2.gazebo.xacro"/>
-<xacro:arg name="mesh_path" default="package://akros2_description/meshes/akros2/" /> <!-- HTTPS URL also works here -->
+<robot name="akros2_mecanum" xmlns:xacro="http://ros.org/wiki/xacro">
+<xacro:include filename="$(find akros2_description)/urdf/akros2_mecanum/akros2_mecanum.common.xacro"/>
+<xacro:include filename="$(find akros2_description)/urdf/akros2_mecanum/akros2_mecanum.control.xacro"/>
+<xacro:include filename="$(find akros2_description)/urdf/akros2_mecanum/akros2_mecanum.gazebo.xacro"/>
+<xacro:arg name="mesh_path" default="package://akros2_description/meshes/akros2_mecanum/" /> <!-- HTTPS URL also works here -->
 <xacro:arg name="unity" default="false" />
 <xacro:property name="mesh_path" value="$(arg mesh_path)" />
@@ -84,28 +84,4 @@
 <!-- IMU_FRAME -->
 <link name="imu_frame"/>
-<!-- T265 TRACKING CAMERA (T265_POSE_FRAME AS WORKAROUND TO KEEP TREE CONTINUOUS)-->
-<link name="t265_pose_frame">
-  <visual>
-    <origin xyz="0 0 0" rpy="0 0 0" />
-    <geometry>
-      <mesh filename="${mesh_path}t265.dae" />
-    </geometry>
-    <material name="Grey"/>
-  </visual>
-  <collision>
-    <origin xyz="0 ${t265_offset_y} 0" rpy="0 0 0" />
-    <geometry>
-      <box size="${t265_length} ${t265_width} ${t265_height}"/>
-    </geometry>
-  </collision>
-</link>
-<!-- T265 TRACKING CAMERA (T265_POSE_INERTIAL)-->
-<link name="t265_pose_inertial">
-  <inertial>
-    <origin xyz="0 0 0" rpy="0 0 0" />
-    <mass value="${t265_mass}" />
-    <xacro:box_inertia m="${t265_mass}" x="${t265_length}" y="${t265_width}" z="${t265_height}"/>
-  </inertial>
-</link>
 <!-- WHEEL LEFT FRONT -->
 <link name="wheel_lf">
@@ -189,16 +165,4 @@
 </link>
 <!-- **** JOINTS **** -->
-<!-- BASE_LINK TO T265_POSE_FRAME -->
-<joint name="pose_base_fixed" type="fixed">
-  <parent link="t265_pose_frame"/>
-  <child link="base_link"/>
-  <origin xyz="${pose_base_offset_x} 0 ${pose_base_offset_z}"/>
-</joint>
-<!-- T265_POSE_INERTIAL TO T265_POSE_FRAME -->
-<joint name="pose_inertial_fixed" type="fixed">
-  <parent link="t265_pose_frame"/>
-  <child link="t265_pose_inertial"/>
-  <origin xyz="0 0 0"/>
-</joint>
 <!-- BASE_LINK_INERTIAL TO BASE_LINK -->
 <joint name="base_inertial_fixed" type="fixed">

File: urdf/akros2_omni/akros2_omni.common.xacro (robot description, xacro)
@@ -1,4 +1,4 @@
 <?xml version="1.0" encoding="utf-8"?>
-<robot name="akros2_common" xmlns:xacro="http://ros.org/wiki/xacro">
+<robot name="omni_common" xmlns:xacro="http://ros.org/wiki/xacro">
 <xacro:property name="pi_by_two" value="1.5707963" />
 <xacro:property name="minus_pi_by_two" value="-1.5707963" />
@@ -19,6 +19,4 @@
 <xacro:property name="wheel_mass" value="0.075" />
 <xacro:property name="wheel_height" value="0.034" />
-<xacro:property name="pose_base_offset_x" value="-0.094" />
-<xacro:property name="pose_base_offset_z" value="-0.115" />
 <xacro:property name="nav_laser_offset_x" value="0.0632" />
 <xacro:property name="laser_frame_offset_z" value="0.0255" />

File: urdf/akros2_omni/akros2_omni.control.xacro (robot description, xacro)
@@ -1,4 +1,4 @@
 <?xml version="1.0" encoding="utf-8"?>
-<robot name="akros2_control" xmlns:xacro="http://ros.org/wiki/xacro">
+<robot name="omni_control" xmlns:xacro="http://ros.org/wiki/xacro">
 <!-- WHEEL_F TRANSMISSION -->
 <transmission name="trans_f">
@@ -12,5 +12,5 @@
   </actuator>
 </transmission>
-<!-- WHEEL_L TRANSMISSION -->
+<!-- WHEEL_L (BACK) TRANSMISSION -->
 <transmission name="trans_l">
   <type>transmission_interface/SimpleTransmission</type>
@@ -23,5 +23,5 @@
   </actuator>
 </transmission>
-<!-- WHEEL_R TRANSMISSION -->
+<!-- WHEEL_R (BACK) TRANSMISSION -->
 <transmission name="trans_r">
   <type>transmission_interface/SimpleTransmission</type>

File: urdf/akros2_omni/akros2_omni.gazebo.xacro (robot description, xacro)
@@ -1,4 +1,4 @@
 <?xml version="1.0" encoding="utf-8"?>
-<robot name="akros2_gazebo" xmlns:xacro="http://ros.org/wiki/xacro">
+<robot name="omni_gazebo" xmlns:xacro="http://ros.org/wiki/xacro">
 <gazebo reference="base_link">
   <material>Gazebo/White</material>

File: urdf/akros2_omni/akros2_omni.urdf (robot description, URDF)
Before this commit: robot akros2, 14 links, 13 joints
Links:
- removed link t265_pose_frame
- removed link t265_pose_inertial
- removed link wheel_lb
- removed link wheel_lf
- removed link wheel_rb
- removed link wheel_rf
- added link wheel_f, mass 0.075; collision cylinder length=0.034 radius=0.038; visual mesh filename=package://akros2_description/meshes/akros2_omni/wheel_f.dae
- added link wheel_l, mass 0.075; collision cylinder length=0.034 radius=0.038; visual mesh filename=package://akros2_description/meshes/akros2_omni/wheel_l.dae
- added link wheel_r, mass 0.075; collision cylinder length=0.034 radius=0.038; visual mesh filename=package://akros2_description/meshes/akros2_omni/wheel_r.dae
Joints:
- removed joint joint_lb
- removed joint joint_lf
- removed joint joint_rb
- removed joint joint_rf
- removed joint pose_base_fixed
- removed joint pose_inertial_fixed
- added joint joint_f: type continuous, parent base_link, child wheel_f, origin xyz=0.0495 0.078 0.021 rpy=0 0 0, axis 0 1 0
- added joint joint_l: type continuous, parent base_link, child wheel_l, origin xyz=-0.0495 0.078 0.021 rpy=0 0 0, axis 0 1 0
- added joint joint_r: type continuous, parent base_link, child wheel_r, origin xyz=0.0495 -0.078 0.021 rpy=0 0 0, axis 0 1 0

File: urdf/akros2_omni/akros2_omni.urdf.xacro (robot description, xacro)
@@ -1,4 +1,4 @@
 <?xml version="1.0" encoding="utf-8"?>
-<robot name="akros2" xmlns:xacro="http://ros.org/wiki/xacro">
+<robot name="akros2_omni" xmlns:xacro="http://ros.org/wiki/xacro">
 <xacro:include filename="$(find akros2_description)/urdf/akros2_omni/akros2_omni.common.xacro"/>
 <xacro:include filename="$(find akros2_description)/urdf/akros2_omni/akros2_omni.control.xacro"/>
@@ -195,5 +195,5 @@
   <axis xyz="0 1 0" />
 </joint>
-<!-- WHEEL_L TO BASE_LINK -->
+<!-- WHEEL_L (BACK) TO BASE_LINK -->
 <joint name="joint_l" type="continuous">
   <parent link="base_link" />
@@ -202,5 +202,5 @@
   <axis xyz="0 1 0" />
 </joint>
-<!-- WHEEL_R TO BASE_LINK -->
+<!-- WHEEL_R (BACK) TO BASE_LINK -->
 <joint name="joint_r" type="continuous">
   <parent link="base_link" />

Commit message: updated base_footprint, imu_link transforms

File: urdf/akros2_mecanum/akros2_mecanum.common.xacro (robot description, xacro)
@@ -1,15 +1,19 @@
 <?xml version="1.0" encoding="utf-8"?>
 <robot name="mecanum_common" xmlns:xacro="http://ros.org/wiki/xacro">
+<!-- All values below are based on CAD model (Fusion 360) -->
 <xacro:property name="pi_by_two" value="1.5707963" />
 <xacro:property name="minus_pi_by_two" value="-1.5707963" />
 <xacro:property name="base_mass" value="2.0" /> <!-- Guesstimate, needs to be measured -->
-<xacro:property name="base_length" value="0.210" />
-<xacro:property name="base_width" value="0.154" /> <!-- Change 0.154 to 0.174 to include motor shafts and emergency button. NB: Geometry intersects wheels -->
+<xacro:property name="base_length" value="0.21038" />
+<xacro:property name="base_width" value="0.1585" /> <!-- Change 0.1585 to 0.2 to include motor shafts and emergency button. NB: Geometry intersects wheels -->
 <xacro:property name="base_height" value="0.099" />
-<xacro:property name="base_offset_x" value="0.003" />
+<xacro:property name="base_offset_x" value="0.00598" />
+<xacro:property name="nav_offset_z" value="-0.099" />
 <xacro:property name="nav_mass" value="0.5" /> <!-- Guesstimate, needs to be measured -->
-<xacro:property name="nav_length" value="0.2" />
-<xacro:property name="nav_width" value="0.154" />
-<xacro:property name="nav_height" value="0.031" />
+<xacro:property name="nav_length" value="0.2004" />
+<xacro:property name="nav_width" value="0.1545" />
+<xacro:property name="nav_height" value="0.03065" />
+<xacro:property name="imu_offset_x" value="0.0562" />
+<xacro:property name="imu_offset_z" value="0.094" />
 <xacro:property name="laser_mass" value="0.12" />
 <xacro:property name="laser_length" value="0.038" />
@@ -19,8 +23,9 @@
 <xacro:property name="wheel_mass" value="0.075" />
 <xacro:property name="wheel_height" value="0.034" />
+<xacro:property name="base_footprint_offset_z" value="-0.015278" />
 <xacro:property name="nav_laser_offset_x" value="0.0632" />
 <xacro:property name="laser_frame_offset_z" value="0.0255" />
 <xacro:property name="joint_offset_x" value="0.0495" />
-<xacro:property name="joint_offset_y" value="0.078" />
+<xacro:property name="joint_offset_y" value="0.08173" />
 <xacro:property name="joint_offset_z" value="0.021" />
 <xacro:macro name="cylinder_inertia" params="m r h">

File: urdf/akros2_mecanum/akros2_mecanum.urdf (robot description, URDF)
Before this commit: robot akros2_mecanum, 12 links, 11 joints
Links:
- link base_link: geometry collision box size=0.21038 0.1585 0.099; visual mesh filename=package://akros2_description/meshes/akros2_mecanum/base_mod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
- link nav_link: geometry collision box size=0.2004 0.1545 0.03065; visual mesh filename=package://akros2_description/meshes/akros2_mecanum/navigati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
Joints:
- joint base_footprint_fixed: origin xyz=0 0 0 -> xyz=0 0 -0.015278
- joint imu_base_fixed: origin xyz=0 0 0 -> xyz=0.0562 0 0.094
- joint joint_lb: origin xyz=-0.0495 0.078 0.021 rpy=0 0 0 -> xyz=-0.0495 0.08173 0.021 rpy=0 0 0
- joint joint_lf: origin xyz=0.0495 0.078 0.021 rpy=0 0 0 -> xyz=0.0495 0.08173 0.021 rpy=0 0 0
- joint joint_rb: origin xyz=-0.0495 -0.078 0.021 rpy=0 0 0 -> xyz=-0.0495 -0.08173 0.021 rpy=0 0 0
- joint joint_rf: origin xyz=0.0495 -0.078 0.021 rpy=0 0 0 -> xyz=0.0495 -0.08173 0.021 rpy=0 0 0

File: urdf/akros2_mecanum/akros2_mecanum.urdf.xacro (robot description, xacro)
@@ -21,5 +21,5 @@
   </visual>
   <collision>
-    <origin xyz="${base_offset_x} 0 ${base_height/2}" rpy="0 0 0" /> <!-- If needed: offset from ground = 0.0278 -->
+    <origin xyz="${base_offset_x/2} 0 ${base_height/2}" rpy="0 0 0" />
     <geometry>
       <box size="${base_length} ${base_width} ${base_height}"/>
@@ -44,5 +44,5 @@
   </inertial>
   <visual>
-    <origin xyz="0 0 -0.099" rpy="0 0 0" />
+    <origin xyz="0 0 ${nav_offset_z}" rpy="0 0 0" />
     <geometry>
       <mesh filename="${mesh_path}navigation_module.dae" />
@@ -51,5 +51,5 @@
   </visual>
   <collision>
-    <origin xyz="0 0 ${nav_height/2}" rpy="0 0 0" /> <!-- If needed: offset from base_link = -0.099 -->
+    <origin xyz="0 0 ${nav_height/2}" rpy="0 0 0" />
     <geometry>
       <box size="${nav_length} ${nav_width} ${nav_height}"/>
@@ -98,5 +98,5 @@
   </visual>
   <collision>
-    <origin xyz="0 ${wheel_height/2} 0" rpy="${pi_by_two} 0 0" /><!-- If needed: offset from joint = 0.01 -->
+    <origin xyz="0 ${wheel_height/2} 0" rpy="${pi_by_two} 0 0" />
     <geometry>
       <cylinder length="${wheel_height}" radius="${wheel_radius}"/>
@@ -118,5 +118,5 @@
   </visual>
   <collision>
-    <origin xyz="0 ${wheel_height/2} 0" rpy="${pi_by_two} 0 0" /><!-- If needed: offset from joint = 0.01 -->
+    <origin xyz="0 ${wheel_height/2} 0" rpy="${pi_by_two} 0 0" />
     <geometry>
       <cylinder length="${wheel_height}" radius="${wheel_radius}"/>
@@ -138,5 +138,5 @@
   </visual>
   <collision>
-    <origin xyz="0 ${-1*(wheel_height/2)} 0" rpy="${pi_by_two} 0 0" /><!-- If needed: offset from joint = 0.01 -->
+    <origin xyz="0 ${-1*(wheel_height/2)} 0" rpy="${pi_by_two} 0 0" />
     <geometry>
       <cylinder length="${wheel_height}" radius="${wheel_radius}"/>
@@ -158,5 +158,5 @@
   </visual>
   <collision>
-    <origin xyz="0 ${-1*(wheel_height/2)} 0" rpy="${pi_by_two} 0 0" /><!-- If needed: offset from joint = 0.01 -->
+    <origin xyz="0 ${-1*(wheel_height/2)} 0" rpy="${pi_by_two} 0 0" />
     <geometry>
       <cylinder length="${wheel_height}" radius="${wheel_radius}"/>
@@ -175,5 +175,5 @@
   <parent link="base_link"/>
   <child link="base_footprint"/>
-  <origin xyz="0 0 0"/>
+  <origin xyz="0 0 ${base_footprint_offset_z}"/>
 </joint>
 <!-- NAV_LINK TO BASE_LINK -->
@@ -200,5 +200,5 @@
   <parent link="base_link"/>
   <child link="imu_link"/>
-  <origin xyz="0 0 0"/>
+  <origin xyz="${imu_offset_x} 0 ${imu_offset_z}"/>
 </joint>
 <!-- IMU_FRAME TO IMU_LINK -->

Commit message: updated urdfs

File: urdf/akros2_mecanum/akros2_mecanum.common.xacro (robot description, xacro)
@@ -44,15 +44,12 @@
             izz="${2*m*r*r/5}" />
 </xacro:macro>
-<material name="FlatBlack">
+<material name="LaserColor">
     <color rgba="0.25 0.25 0.25 1"/>
 </material>
-<material name="DarkGrey">
+<material name="WheelsNavColor">
+    <color rgba="0.35 0.35 0.35 1"/>
+</material>
+<material name="BaseLinkColor">
     <color rgba="0.5 0.5 0.5 1"/>
 </material>
-<material name="Grey">
-    <color rgba="0.75 0.75 0.75 1"/>
-</material>
-<material name="White">
-     <color rgba="1 1 1 1"/>
-</material>
 </robot>

File: urdf/akros2_mecanum/akros2_mecanum.gazebo.xacro (robot description, xacro)
@@ -2,5 +2,5 @@
 <robot name="mecanum_gazebo" xmlns:xacro="http://ros.org/wiki/xacro">
 <gazebo reference="base_link">
-  <material>Gazebo/White</material>
+  <material>Gazebo/Grey</material>
 </gazebo>
 <gazebo reference="nav_link">

File: urdf/akros2_mecanum/akros2_mecanum.urdf.xacro (robot description, xacro)
@@ -18,5 +18,5 @@
       <mesh filename="${mesh_path}base_module.dae" />
     </geometry>
-   <material name="White"/>
+   <material name="BaseLinkColor"/>
   </visual>
   <collision>
@@ -48,5 +48,5 @@
       <mesh filename="${mesh_path}navigation_module.dae" />
     </geometry>
-    <material name="DarkGrey"/>
+    <material name="WheelsNavColor"/>
   </visual>
   <collision>
@@ -69,5 +69,5 @@
       <mesh filename="${mesh_path}ld06.dae" />
     </geometry>
-    <material name="FlatBlack"/>
+    <material name="LaserColor"/>
   </visual>
   <collision>
@@ -95,5 +95,5 @@
       <mesh filename="${mesh_path}wheel_lf.dae" />
     </geometry>
-    <material name="FlatBlack"/>
+    <material name="WheelsNavColor"/>
   </visual>
   <collision>
@@ -115,5 +115,5 @@
       <mesh filename="${mesh_path}wheel_lb.dae" />
     </geometry>
-    <material name="FlatBlack"/>
+    <material name="WheelsNavColor"/>
   </visual>
   <collision>
@@ -135,5 +135,5 @@
       <mesh filename="${mesh_path}wheel_rf.dae" />
     </geometry>
-    <material name="FlatBlack"/>
+    <material name="WheelsNavColor"/>
   </visual>
   <collision>
@@ -155,5 +155,5 @@
       <mesh filename="${mesh_path}wheel_rb.dae" />
     </geometry>
-    <material name="FlatBlack"/>
+    <material name="WheelsNavColor"/>
   </visual>
   <collision>

Commit message: updated base link translucense

File: urdf/akros2_mecanum/akros2_mecanum.common.xacro (robot description, xacro)
@@ -5,8 +5,8 @@
 <xacro:property name="minus_pi_by_two" value="-1.5707963" />
 <xacro:property name="base_mass" value="2.0" /> <!-- Guesstimate, needs to be measured -->
-<xacro:property name="base_length" value="0.21038" />
+<xacro:property name="base_length" value="0.2104" />
 <xacro:property name="base_width" value="0.1585" /> <!-- Change 0.1585 to 0.2 to include motor shafts and emergency button. NB: Geometry intersects wheels -->
 <xacro:property name="base_height" value="0.099" />
-<xacro:property name="base_offset_x" value="0.00598" />
+<xacro:property name="base_offset_x" value="0.006" />
 <xacro:property name="nav_offset_z" value="-0.099" />
 <xacro:property name="nav_mass" value="0.5" /> <!-- Guesstimate, needs to be measured -->
@@ -51,5 +51,5 @@
 </material>
 <material name="BaseLinkColor">
-    <color rgba="0.5 0.5 0.5 1"/>
+    <color rgba="0.5 0.5 0.5 0.95"/>
 </material>
 </robot>

Commit message: Update akros2_mecanum.common.xacro

File: urdf/akros2_mecanum/akros2_mecanum.common.xacro (robot description, xacro)
@@ -5,6 +5,6 @@
 <xacro:property name="minus_pi_by_two" value="-1.5707963" />
 <xacro:property name="base_mass" value="2.0" /> <!-- Guesstimate, needs to be measured -->
-<xacro:property name="base_length" value="0.2104" />
-<xacro:property name="base_width" value="0.1585" /> <!-- Change 0.1585 to 0.2 to include motor shafts and emergency button. NB: Geometry intersects wheels -->
+<xacro:property name="base_length" value="0.2104" /> <!-- Change 0.2064 to 0.2104 to include screw heads in collision. -->
+<xacro:property name="base_width" value="0.1585" /> <!-- Change 0.1585 to 0.2 to include motor shafts and emergency button in collision. Note: Geometry intersects wheels -->
 <xacro:property name="base_height" value="0.099" />
 <xacro:property name="base_offset_x" value="0.006" />

Commit message: Update akros2_mecanum.common.xacro

File: urdf/akros2_mecanum/akros2_mecanum.common.xacro (robot description, xacro)
@@ -5,5 +5,5 @@
 <xacro:property name="minus_pi_by_two" value="-1.5707963" />
 <xacro:property name="base_mass" value="2.0" /> <!-- Guesstimate, needs to be measured -->
-<xacro:property name="base_length" value="0.2104" /> <!-- Change 0.2064 to 0.2104 to include screw heads in collision. -->
+<xacro:property name="base_length" value="0.20638" /> <!-- Change 0.20638 to 0.21038 to include screw heads in collision. -->
 <xacro:property name="base_width" value="0.1585" /> <!-- Change 0.1585 to 0.2 to include motor shafts and emergency button in collision. Note: Geometry intersects wheels -->
 <xacro:property name="base_height" value="0.099" />

Commit message: Update akros2_mecanum.common.xacro

File: urdf/akros2_mecanum/akros2_mecanum.common.xacro (robot description, xacro)
@@ -20,7 +20,7 @@
 <xacro:property name="laser_width" value="0.0381" />
 <xacro:property name="laser_height" value="0.033" />
-<xacro:property name="wheel_radius" value="0.038" />
-<xacro:property name="wheel_mass" value="0.075" />
-<xacro:property name="wheel_height" value="0.034" />
+<xacro:property name="wheel_radius" value="0.036" /> <!-- Actual radius is 0.0385 -->
+<xacro:property name="wheel_mass" value="0.075" /> <!-- Guesstimate, needs to be measured -->
+<xacro:property name="wheel_height" value="0.0315" /> <!-- Actual height is 0.034 -->
 <xacro:property name="base_footprint_offset_z" value="-0.015278" />
 <xacro:property name="nav_laser_offset_x" value="0.0632" />

Commit message: Update akros2_mecanum.common.xacro

File: urdf/akros2_mecanum/akros2_mecanum.common.xacro (robot description, xacro)
@@ -27,5 +27,5 @@
 <xacro:property name="laser_frame_offset_z" value="0.0255" />
 <xacro:property name="joint_offset_x" value="0.0495" />
-<xacro:property name="joint_offset_y" value="0.08173" />
+<xacro:property name="joint_offset_y" value="0.0854225" />
 <xacro:property name="joint_offset_z" value="0.021" />
 <xacro:macro name="cylinder_inertia" params="m r h">

Commit message: Update akros2_mecanum.common.xacro

File: urdf/akros2_mecanum/akros2_mecanum.common.xacro (robot description, xacro)
@@ -23,5 +23,5 @@
 <xacro:property name="wheel_mass" value="0.075" /> <!-- Guesstimate, needs to be measured -->
 <xacro:property name="wheel_height" value="0.0315" /> <!-- Actual height is 0.034 -->
-<xacro:property name="base_footprint_offset_z" value="-0.015278" />
+<xacro:property name="base_footprint_offset_z" value="-0.015377" /> <!-- Actual offset is -0.017877 -->
 <xacro:property name="nav_laser_offset_x" value="0.0632" />
 <xacro:property name="laser_frame_offset_z" value="0.0255" />
