Commit message: Update akros2_mecanum.common.xacro

File: urdf/akros2_mecanum/akros2_mecanum.common.xacro (robot description, xacro)
@@ -6,5 +6,5 @@
 <xacro:property name="base_mass" value="2.0" /> <!-- Guesstimate, needs to be measured -->
 <xacro:property name="base_length" value="0.20638" /> <!-- Change 0.20638 to 0.21038 to include screw heads in collision. -->
-<xacro:property name="base_width" value="0.1585" /> <!-- Change 0.1585 to 0.2 to include motor shafts and emergency button in collision. Note: Geometry intersects wheels -->
+<xacro:property name="base_width" value="0.1545" /> <!-- Change 0.1545 to 0.1585 to include screw heads in collision, and to 0.2 to include motor shafts and emergency button in collision.-->
 <xacro:property name="base_height" value="0.099" />
 <xacro:property name="base_offset_x" value="0.006" />

Commit message: Update akros2_mecanum.common.xacro

File: urdf/akros2_mecanum/akros2_mecanum.common.xacro (robot description, xacro)
@@ -6,5 +6,5 @@
 <xacro:property name="base_mass" value="2.0" /> <!-- Guesstimate, needs to be measured -->
 <xacro:property name="base_length" value="0.20638" /> <!-- Change 0.20638 to 0.21038 to include screw heads in collision. -->
-<xacro:property name="base_width" value="0.1545" /> <!-- Change 0.1545 to 0.1585 to include screw heads in collision, and to 0.2 to include motor shafts and emergency button in collision.-->
+<xacro:property name="base_width" value="0.1545" /> <!-- Change 0.1545 to 0.1585 to include screw heads in collision, and to 0.2 to include motor shafts and emergency button (Geometry intersects wheels).-->
 <xacro:property name="base_height" value="0.099" />
 <xacro:property name="base_offset_x" value="0.006" />

Commit message: Update akros2_mecanum.common.xacro

File: urdf/akros2_mecanum/akros2_mecanum.common.xacro (robot description, xacro)
@@ -6,5 +6,5 @@
 <xacro:property name="base_mass" value="2.0" /> <!-- Guesstimate, needs to be measured -->
 <xacro:property name="base_length" value="0.20638" /> <!-- Change 0.20638 to 0.21038 to include screw heads in collision. -->
-<xacro:property name="base_width" value="0.1545" /> <!-- Change 0.1545 to 0.1585 to include screw heads in collision, and to 0.2 to include motor shafts and emergency button (Geometry intersects wheels).-->
+<xacro:property name="base_width" value="0.1565" /> <!-- Actual width = 0.1545 (2mm added as offset). Change 0.1565 to 0.2 to include motor shafts and emergency button (Geometry intersects wheels).-->
 <xacro:property name="base_height" value="0.099" />
 <xacro:property name="base_offset_x" value="0.006" />

Commit message: Update akros2_mecanum.common.xacro

File: urdf/akros2_mecanum/akros2_mecanum.common.xacro (robot description, xacro)
@@ -6,5 +6,5 @@
 <xacro:property name="base_mass" value="2.0" /> <!-- Guesstimate, needs to be measured -->
 <xacro:property name="base_length" value="0.20638" /> <!-- Change 0.20638 to 0.21038 to include screw heads in collision. -->
-<xacro:property name="base_width" value="0.1565" /> <!-- Actual width = 0.1545 (2mm added as offset). Change 0.1565 to 0.2 to include motor shafts and emergency button (Geometry intersects wheels).-->
+<xacro:property name="base_width" value="0.1565" /> <!-- Actual width = 0.1545 without screw heads (2mm added as offset). Change 0.1565 to 0.2 to include motor shafts and emergency button (Geometry intersects wheels).-->
 <xacro:property name="base_height" value="0.099" />
 <xacro:property name="base_offset_x" value="0.006" />
@@ -12,5 +12,5 @@
 <xacro:property name="nav_mass" value="0.5" /> <!-- Guesstimate, needs to be measured -->
 <xacro:property name="nav_length" value="0.2004" />
-<xacro:property name="nav_width" value="0.1545" />
+<xacro:property name="nav_width" value="0.1565" /> <!-- Actual width = 0.1545 (2mm added as offset).-->
 <xacro:property name="nav_height" value="0.03065" />
 <xacro:property name="imu_offset_x" value="0.0562" />

Commit message: Update akros2_mecanum.common.xacro

File: urdf/akros2_mecanum/akros2_mecanum.common.xacro (robot description, xacro)
@@ -5,6 +5,6 @@
 <xacro:property name="minus_pi_by_two" value="-1.5707963" />
 <xacro:property name="base_mass" value="2.0" /> <!-- Guesstimate, needs to be measured -->
-<xacro:property name="base_length" value="0.20638" /> <!-- Change 0.20638 to 0.21038 to include screw heads in collision. -->
-<xacro:property name="base_width" value="0.1565" /> <!-- Actual width = 0.1545 without screw heads (2mm added as offset). Change 0.1565 to 0.2 to include motor shafts and emergency button (Geometry intersects wheels).-->
+<xacro:property name="base_length" value="0.20638" /> <!-- Actual length = 0.20638 (1mm added on both sides as padding). Change 0.20638 to 0.21038 to include screw heads in collision. -->
+<xacro:property name="base_width" value="0.1565" /> <!-- Actual width = 0.1545 without screw heads (1mm added on both sides as padding). Change 0.1565 to 0.2 to include motor shafts and emergency button (Geometry intersects wheels).-->
 <xacro:property name="base_height" value="0.099" />
 <xacro:property name="base_offset_x" value="0.006" />
@@ -12,5 +12,5 @@
 <xacro:property name="nav_mass" value="0.5" /> <!-- Guesstimate, needs to be measured -->
 <xacro:property name="nav_length" value="0.2004" />
-<xacro:property name="nav_width" value="0.1565" /> <!-- Actual width = 0.1545 (2mm added as offset).-->
+<xacro:property name="nav_width" value="0.1565" /> <!-- Actual width = 0.1545 (1mm added on both sides as offset).-->
 <xacro:property name="nav_height" value="0.03065" />
 <xacro:property name="imu_offset_x" value="0.0562" />

Commit message: Update akros2_mecanum.common.xacro

File: urdf/akros2_mecanum/akros2_mecanum.common.xacro (robot description, xacro)
@@ -5,5 +5,5 @@
 <xacro:property name="minus_pi_by_two" value="-1.5707963" />
 <xacro:property name="base_mass" value="2.0" /> <!-- Guesstimate, needs to be measured -->
-<xacro:property name="base_length" value="0.20638" /> <!-- Actual length = 0.20638 (1mm added on both sides as padding). Change 0.20638 to 0.21038 to include screw heads in collision. -->
+<xacro:property name="base_length" value="0.20838" /> <!-- Actual length = 0.20638 (1mm added on both sides as padding). Change 0.20638 to 0.21038 to include screw heads in collision. -->
 <xacro:property name="base_width" value="0.1565" /> <!-- Actual width = 0.1545 without screw heads (1mm added on both sides as padding). Change 0.1565 to 0.2 to include motor shafts and emergency button (Geometry intersects wheels).-->
 <xacro:property name="base_height" value="0.099" />

Commit message: Update akros2_mecanum.common.xacro

File: urdf/akros2_mecanum/akros2_mecanum.common.xacro (robot description, xacro)
@@ -1,10 +1,10 @@
 <?xml version="1.0" encoding="utf-8"?>
 <robot name="mecanum_common" xmlns:xacro="http://ros.org/wiki/xacro">
-<!-- All values below are based on CAD model (Fusion 360) -->
+<!-- All values below are based on CAD model (Fusion 360). 1mm added on each side - length, width (2mm total) as padding. -->
 <xacro:property name="pi_by_two" value="1.5707963" />
 <xacro:property name="minus_pi_by_two" value="-1.5707963" />
 <xacro:property name="base_mass" value="2.0" /> <!-- Guesstimate, needs to be measured -->
-<xacro:property name="base_length" value="0.20838" /> <!-- Actual length = 0.20638 (1mm added on both sides as padding). Change 0.20638 to 0.21038 to include screw heads in collision. -->
-<xacro:property name="base_width" value="0.1565" /> <!-- Actual width = 0.1545 without screw heads (1mm added on both sides as padding). Change 0.1565 to 0.2 to include motor shafts and emergency button (Geometry intersects wheels).-->
+<xacro:property name="base_length" value="0.20838" /> <!-- Actual length = 0.20638. Change 0.20638 to 0.21038 to include screw heads in collision. -->
+<xacro:property name="base_width" value="0.1565" /> <!-- Actual width = 0.1545 without screw heads. Change 0.1565 to 0.2 to include motor shafts and emergency button (Geometry intersects wheels).-->
 <xacro:property name="base_height" value="0.099" />
 <xacro:property name="base_offset_x" value="0.006" />

Commit message: Update akros2_mecanum.common.xacro

File: urdf/akros2_mecanum/akros2_mecanum.common.xacro (robot description, xacro)
@@ -1,5 +1,5 @@
 <?xml version="1.0" encoding="utf-8"?>
 <robot name="mecanum_common" xmlns:xacro="http://ros.org/wiki/xacro">
-<!-- All values below are based on CAD model (Fusion 360). 1mm added on each side - length, width (2mm total) as padding. -->
+<!-- All values below are based on CAD model (Fusion 360). 1mm added on each side (2mm total) for length, width (but not height) as padding. -->
 <xacro:property name="pi_by_two" value="1.5707963" />
 <xacro:property name="minus_pi_by_two" value="-1.5707963" />
@@ -20,8 +20,8 @@
 <xacro:property name="laser_width" value="0.0381" />
 <xacro:property name="laser_height" value="0.033" />
-<xacro:property name="wheel_radius" value="0.036" /> <!-- Actual radius is 0.0385 -->
+<xacro:property name="wheel_radius" value="0.036" /> <!-- Actual radius = 0.0385 -->
 <xacro:property name="wheel_mass" value="0.075" /> <!-- Guesstimate, needs to be measured -->
-<xacro:property name="wheel_height" value="0.0315" /> <!-- Actual height is 0.034 -->
-<xacro:property name="base_footprint_offset_z" value="-0.015377" /> <!-- Actual offset is -0.017877 -->
+<xacro:property name="wheel_width" value="0.0335" /> <!-- CAD width without padding = 0.0315, Actual width without padding = 0.034 -->
+<xacro:property name="base_footprint_offset_z" value="-0.015377" /> <!-- Actual offset = -0.017877 -->
 <xacro:property name="nav_laser_offset_x" value="0.0632" />
 <xacro:property name="laser_frame_offset_z" value="0.0255" />

Commit message: Update akros2_mecanum.common.xacro

File: urdf/akros2_mecanum/akros2_mecanum.common.xacro (robot description, xacro)
@@ -5,6 +5,6 @@
 <xacro:property name="minus_pi_by_two" value="-1.5707963" />
 <xacro:property name="base_mass" value="2.0" /> <!-- Guesstimate, needs to be measured -->
-<xacro:property name="base_length" value="0.20838" /> <!-- Actual length = 0.20638. Change 0.20638 to 0.21038 to include screw heads in collision. -->
-<xacro:property name="base_width" value="0.1565" /> <!-- Actual width = 0.1545 without screw heads. Change 0.1565 to 0.2 to include motor shafts and emergency button (Geometry intersects wheels).-->
+<xacro:property name="base_length" value="0.20838" /> <!-- Actual length without padding = 0.20638. Change 0.20638 to 0.21038 to include screw heads in collision. -->
+<xacro:property name="base_width" value="0.1565" /> <!-- Actual width without padding = 0.1545 without screw heads. Change 0.1565 to 0.2 to include motor shafts and emergency button (Geometry intersects wheels).-->
 <xacro:property name="base_height" value="0.099" />
 <xacro:property name="base_offset_x" value="0.006" />
@@ -12,5 +12,5 @@
 <xacro:property name="nav_mass" value="0.5" /> <!-- Guesstimate, needs to be measured -->
 <xacro:property name="nav_length" value="0.2004" />
-<xacro:property name="nav_width" value="0.1565" /> <!-- Actual width = 0.1545 (1mm added on both sides as offset).-->
+<xacro:property name="nav_width" value="0.1565" /> <!-- Actual width without padding = 0.1545-->
 <xacro:property name="nav_height" value="0.03065" />
 <xacro:property name="imu_offset_x" value="0.0562" />
@@ -22,5 +22,5 @@
 <xacro:property name="wheel_radius" value="0.036" /> <!-- Actual radius = 0.0385 -->
 <xacro:property name="wheel_mass" value="0.075" /> <!-- Guesstimate, needs to be measured -->
-<xacro:property name="wheel_width" value="0.0335" /> <!-- CAD width without padding = 0.0315, Actual width without padding = 0.034 -->
+<xacro:property name="wheel_thickness" value="0.034" /> <!-- Actual thickness = 0.034. CAD thickness = 0.0315 -->
 <xacro:property name="base_footprint_offset_z" value="-0.015377" /> <!-- Actual offset = -0.017877 -->
 <xacro:property name="nav_laser_offset_x" value="0.0632" />

Commit message: Update akros2_mecanum.common.xacro

File: urdf/akros2_mecanum/akros2_mecanum.common.xacro (robot description, xacro)
@@ -20,7 +20,7 @@
 <xacro:property name="laser_width" value="0.0381" />
 <xacro:property name="laser_height" value="0.033" />
-<xacro:property name="wheel_radius" value="0.036" /> <!-- Actual radius = 0.0385 -->
+<xacro:property name="wheel_radius" value="0.0385" /> <!-- Actual radius = 0.0385, CAD radius = 0.036 -->
 <xacro:property name="wheel_mass" value="0.075" /> <!-- Guesstimate, needs to be measured -->
-<xacro:property name="wheel_thickness" value="0.034" /> <!-- Actual thickness = 0.034. CAD thickness = 0.0315 -->
+<xacro:property name="wheel_thickness" value="0.034" /> <!-- Actual thickness = 0.034, CAD thickness = 0.0315 -->
 <xacro:property name="base_footprint_offset_z" value="-0.015377" /> <!-- Actual offset = -0.017877 -->
 <xacro:property name="nav_laser_offset_x" value="0.0632" />

Commit message: Update akros2_mecanum.common.xacro

File: urdf/akros2_mecanum/akros2_mecanum.common.xacro (robot description, xacro)
@@ -23,5 +23,5 @@
 <xacro:property name="wheel_mass" value="0.075" /> <!-- Guesstimate, needs to be measured -->
 <xacro:property name="wheel_thickness" value="0.034" /> <!-- Actual thickness = 0.034, CAD thickness = 0.0315 -->
-<xacro:property name="base_footprint_offset_z" value="-0.015377" /> <!-- Actual offset = -0.017877 -->
+<xacro:property name="base_footprint_offset_z" value="-0.015377" /> <!-- Actual offset = -0.017877, CAD offset = -0.015377 -->
 <xacro:property name="nav_laser_offset_x" value="0.0632" />
 <xacro:property name="laser_frame_offset_z" value="0.0255" />

Commit message: Update akros2_mecanum.common.xacro

File: urdf/akros2_mecanum/akros2_mecanum.common.xacro (robot description, xacro)
@@ -23,5 +23,5 @@
 <xacro:property name="wheel_mass" value="0.075" /> <!-- Guesstimate, needs to be measured -->
 <xacro:property name="wheel_thickness" value="0.034" /> <!-- Actual thickness = 0.034, CAD thickness = 0.0315 -->
-<xacro:property name="base_footprint_offset_z" value="-0.015377" /> <!-- Actual offset = -0.017877, CAD offset = -0.015377 -->
+<xacro:property name="base_footprint_offset_z" value="-0.017877" /> <!-- Actual offset = -0.017877, CAD offset = -0.015377 -->
 <xacro:property name="nav_laser_offset_x" value="0.0632" />
 <xacro:property name="laser_frame_offset_z" value="0.0255" />

Commit message: Update akros2_mecanum.common.xacro

File: urdf/akros2_mecanum/akros2_mecanum.common.xacro (robot description, xacro)
@@ -5,6 +5,6 @@
 <xacro:property name="minus_pi_by_two" value="-1.5707963" />
 <xacro:property name="base_mass" value="2.0" /> <!-- Guesstimate, needs to be measured -->
-<xacro:property name="base_length" value="0.20838" /> <!-- Actual length without padding = 0.20638. Change 0.20638 to 0.21038 to include screw heads in collision. -->
-<xacro:property name="base_width" value="0.1565" /> <!-- Actual width without padding = 0.1545 without screw heads. Change 0.1565 to 0.2 to include motor shafts and emergency button (Geometry intersects wheels).-->
+<xacro:property name="base_length" value="0.20838" /> <!-- Actual length without padding = 0.20638. Change to 0.21038 to include screw heads in collision (without padding). -->
+<xacro:property name="base_width" value="0.1565" /> <!-- Actual width without padding = 0.1545 without screw heads. Change to 0.2 to include motor shafts and emergency button (without padding)-->
 <xacro:property name="base_height" value="0.099" />
 <xacro:property name="base_offset_x" value="0.006" />

Commit message: Update akros2_mecanum.common.xacro

File: urdf/akros2_mecanum/akros2_mecanum.common.xacro (robot description, xacro)
@@ -11,5 +11,5 @@
 <xacro:property name="nav_offset_z" value="-0.099" />
 <xacro:property name="nav_mass" value="0.5" /> <!-- Guesstimate, needs to be measured -->
-<xacro:property name="nav_length" value="0.2004" />
+<xacro:property name="nav_length" value="0.2024" /> <!-- Actual length without padding = 0.2004 -->
 <xacro:property name="nav_width" value="0.1565" /> <!-- Actual width without padding = 0.1545-->
 <xacro:property name="nav_height" value="0.03065" />

Commit message: Update akros2_mecanum.common.xacro

File: urdf/akros2_mecanum/akros2_mecanum.common.xacro (robot description, xacro)
@@ -17,6 +17,6 @@
 <xacro:property name="imu_offset_z" value="0.094" />
 <xacro:property name="laser_mass" value="0.12" />
-<xacro:property name="laser_length" value="0.038" />
-<xacro:property name="laser_width" value="0.0381" />
+<xacro:property name="laser_length" value="0.04" /> <!-- Actual length without padding = 0.038 -->
+<xacro:property name="laser_width" value="0.0401" /> <!-- Actual width without padding = 0.0381 -->
 <xacro:property name="laser_height" value="0.033" />
 <xacro:property name="wheel_radius" value="0.0385" /> <!-- Actual radius = 0.0385, CAD radius = 0.036 -->

Commit message: Update akros2_mecanum.common.xacro

File: urdf/akros2_mecanum/akros2_mecanum.common.xacro (robot description, xacro)
@@ -1,22 +1,22 @@
 <?xml version="1.0" encoding="utf-8"?>
 <robot name="mecanum_common" xmlns:xacro="http://ros.org/wiki/xacro">
-<!-- All values below are based on CAD model (Fusion 360). 1mm added on each side (2mm total) for length and width (but not height) as padding. -->
+<!-- All values below are based on CAD model (Fusion 360). 2mm added on each side (4mm total) for length and width (but not height) as padding. -->
 <xacro:property name="pi_by_two" value="1.5707963" />
 <xacro:property name="minus_pi_by_two" value="-1.5707963" />
 <xacro:property name="base_mass" value="2.0" /> <!-- Guesstimate, needs to be measured -->
-<xacro:property name="base_length" value="0.20838" /> <!-- Actual length without padding = 0.20638. Change to 0.21038 to include screw heads in collision (without padding). -->
-<xacro:property name="base_width" value="0.1565" /> <!-- Actual width without padding = 0.1545 without screw heads. Change to 0.2 to include motor shafts and emergency button (without padding)-->
+<xacro:property name="base_length" value="0.21038" /> <!-- Actual length without padding = 0.20638. Change to 0.21038 to include screw heads in collision (without padding). -->
+<xacro:property name="base_width" value="0.1585" /> <!-- Actual width without padding = 0.1545 without screw heads. Change to 0.2 to include motor shafts and emergency button (without padding)-->
 <xacro:property name="base_height" value="0.099" />
 <xacro:property name="base_offset_x" value="0.006" />
 <xacro:property name="nav_offset_z" value="-0.099" />
 <xacro:property name="nav_mass" value="0.5" /> <!-- Guesstimate, needs to be measured -->
-<xacro:property name="nav_length" value="0.2024" /> <!-- Actual length without padding = 0.2004 -->
-<xacro:property name="nav_width" value="0.1565" /> <!-- Actual width without padding = 0.1545-->
+<xacro:property name="nav_length" value="0.2044" /> <!-- Actual length without padding = 0.2004 -->
+<xacro:property name="nav_width" value="0.1585" /> <!-- Actual width without padding = 0.1545-->
 <xacro:property name="nav_height" value="0.03065" />
 <xacro:property name="imu_offset_x" value="0.0562" />
 <xacro:property name="imu_offset_z" value="0.094" />
 <xacro:property name="laser_mass" value="0.12" />
-<xacro:property name="laser_length" value="0.04" /> <!-- Actual length without padding = 0.038 -->
-<xacro:property name="laser_width" value="0.0401" /> <!-- Actual width without padding = 0.0381 -->
+<xacro:property name="laser_length" value="0.042" /> <!-- Actual length without padding = 0.038 -->
+<xacro:property name="laser_width" value="0.0421" /> <!-- Actual width without padding = 0.0381 -->
 <xacro:property name="laser_height" value="0.033" />
 <xacro:property name="wheel_radius" value="0.0385" /> <!-- Actual radius = 0.0385, CAD radius = 0.036 -->
