Commit message: Update akros2_mecanum.urdf

File: urdf/akros2_mecanum/akros2_mecanum.urdf (robot description, URDF)
Before this commit: robot akros2_mecanum, 12 links, 11 joints
Links:
- link base_link: geometry collision box size=0.2064 0.1585 0.099; visual mesh filename=package://akros2_description/meshes/akros2_mecanum/base_mod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

Commit message: Update akros2_mecanum.urdf

File: urdf/akros2_mecanum/akros2_mecanum.urdf (robot description, URDF)
Before this commit: robot akros2_mecanum, 12 links, 11 joints
Links:
- link base_link: geometry collision box size=0.20638 0.1585 0.099; visual mesh filename=package://akros2_description/meshes/akros2_mecanum/base_mod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

Commit message: Update akros2_mecanum.urdf

File: urdf/akros2_mecanum/akros2_mecanum.urdf (robot description, URDF)
Before this commit: robot akros2_mecanum, 12 links, 11 joints
Links:
- link wheel_lb: geometry collision cylinder length=0.0315 radius=0.038; visual mesh filename=package://akros2_description/meshes/akros2_mecanum/wheel_lb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
- link wheel_lf: geometry collision cylinder length=0.0315 radius=0.038; visual mesh filename=package://akros2_description/meshes/akros2_mecanum/wheel_lf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
- link wheel_rb: geometry collision cylinder length=0.0315 radius=0.038; visual mesh filename=package://akros2_description/meshes/akros2_mecanum/wheel_rb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
- link wheel_rf: geometry collision cylinder length=0.0315 radius=0.038; visual mesh filename=package://akros2_description/meshes/akros2_mecanum/wheel_rf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

Commit message: Update akros2_mecanum.urdf

File: urdf/akros2_mecanum/akros2_mecanum.urdf (robot description, URDF)
Before this commit: robot akros2_mecanum, 12 links, 11 joints
Links:
- link wheel_lb: geometry collision cylinder length=0.0315 radius=0.036; visual mesh filename=package://akros2_description/meshes/akros2_mecanum/wheel_lb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
- link wheel_lf: geometry collision cylinder length=0.0315 radius=0.036; visual mesh filename=package://akros2_description/meshes/akros2_mecanum/wheel_lf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
- link wheel_rb: geometry collision cylinder length=0.0315 radius=0.036; visual mesh filename=package://akros2_description/meshes/akros2_mecanum/wheel_rb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
- link wheel_rf: geometry collision cylinder length=0.0315 radius=0.036; visual mesh filename=package://akros2_description/meshes/akros2_mecanum/wheel_rf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

Commit message: Update akros2_mecanum.urdf

File: urdf/akros2_mecanum/akros2_mecanum.urdf (robot description, URDF)
Before this commit: robot akros2_mecanum, 12 links, 11 joints
Links:
- link base_link: geometry collision box size=0.20838 0.1565 0.099; visual mesh filename=package://akros2_description/meshes/akros2_mecanum/base_mod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
- link nav_link: geometry collision box size=0.2024 0.1565 0.03065; visual mesh filename=package://akros2_description/meshes/akros2_mecanum/navigati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
- link wheel_lb: geometry collision cylinder length=0.034 radius=0.0385; visual mesh filename=package://akros2_description/meshes/akros2_mecanum/wheel_lb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
- link wheel_lf: geometry collision cylinder length=0.034 radius=0.0385; visual mesh filename=package://akros2_description/meshes/akros2_mecanum/wheel_lf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
- link wheel_rb: geometry collision cylinder length=0.034 radius=0.0385; visual mesh filename=package://akros2_description/meshes/akros2_mecanum/wheel_rb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
- link wheel_rf: geometry collision cylinder length=0.034 radius=0.0385; visual mesh filename=package://akros2_description/meshes/akros2_mecanum/wheel_rf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
Joints:
- joint base_footprint_fixed: origin xyz=0 0 -0.015278 -> xyz=0 0 -0.017877
- joint joint_lb: origin xyz=-0.0495 0.08173 0.021 rpy=0 0 0 -> xyz=-0.0495 0.0854225 0.021 rpy=0 0 0
- joint joint_lf: origin xyz=0.0495 0.08173 0.021 rpy=0 0 0 -> xyz=0.0495 0.0854225 0.021 rpy=0 0 0
- joint joint_rb: origin xyz=-0.0495 -0.08173 0.021 rpy=0 0 0 -> xyz=-0.0495 -0.0854225 0.021 rpy=0 0 0
- joint joint_rf: origin xyz=0.0495 -0.08173 0.021 rpy=0 0 0 -> xyz=0.0495 -0.0854225 0.021 rpy=0 0 0

Commit message: Update akros2_mecanum.urdf

File: urdf/akros2_mecanum/akros2_mecanum.urdf (robot description, URDF)
Before this commit: robot akros2_mecanum, 12 links, 11 joints
Links:
- link laser_link: geometry collision box size=0.04 0.0401 0.033; visual mesh filename=package://akros2_description/meshes/akros2_mecanum/ld06.dae

Commit message: Update akros2_mecanum.urdf

File: urdf/akros2_mecanum/akros2_mecanum.urdf (robot description, URDF)
Before this commit: robot akros2_mecanum, 12 links, 11 joints
Links:
- link base_link: geometry collision box size=0.21038 0.1585 0.099; visual mesh filename=package://akros2_description/meshes/akros2_mecanum/base_mod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
- link laser_link: geometry collision box size=0.042 0.0421 0.033; visual mesh filename=package://akros2_description/meshes/akros2_mecanum/ld06.dae
- link nav_link: geometry collision box size=0.2044 0.1585 0.03065; visual mesh filename=package://akros2_description/meshes/akros2_mecanum/navigati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
