Commit message: update urdf - set base_footprint as parent of base_link

File: urdf/akros2_mecanum/robot.gazebo.xacro (robot description, xacro)
@@ -1,6 +1,6 @@
 <?xml version="1.0" encoding="utf-8"?>
-<robot name="omni_gazebo" xmlns:xacro="http://ros.org/wiki/xacro">
+<robot name="mecanum_gazebo" xmlns:xacro="http://ros.org/wiki/xacro">
 <gazebo reference="base_link">
-  <material>Gazebo/White</material>
+  <material>Gazebo/Grey</material>
 </gazebo>
 <gazebo reference="nav_link">
@@ -10,11 +10,14 @@
   <material>Gazebo/FlatBlack</material>
 </gazebo>
-<gazebo reference="wheel_f">
+<gazebo reference="wheel_lf">
   <material>Gazebo/DarkGrey</material>
 </gazebo>
-<gazebo reference="wheel_l">
+<gazebo reference="wheel_lb">
   <material>Gazebo/DarkGrey</material>
 </gazebo>
-<gazebo reference="wheel_r">
+<gazebo reference="wheel_rf">
+  <material>Gazebo/DarkGrey</material>
+</gazebo>
+<gazebo reference="wheel_rb">
   <material>Gazebo/DarkGrey</material>
 </gazebo>
@@ -84,5 +87,5 @@
     <odometryFrame>odom</odometryFrame>
     <odometryRate>100.0</odometryRate>
-    <robotBaseFrame>base_link</robotBaseFrame>
+    <robotBaseFrame>base_footprint</robotBaseFrame>
     <publishTF>false</publishTF>
   </plugin>

File: urdf/akros2_mecanum/robot.urdf (robot description, URDF)
Before this commit: robot akros2_mecanum, 12 links, 11 joints
Joints:
- removed joint base_footprint_fixed
- added joint footprint_base_fixed: type fixed, parent base_footprint, child base_link, origin xyz=0 0 0.017877

File: urdf/akros2_mecanum/robot.urdf.xacro (robot description, xacro)
@@ -1,7 +1,7 @@
 <?xml version="1.0" encoding="utf-8"?>
 <robot name="akros2_mecanum" xmlns:xacro="http://ros.org/wiki/xacro">
-<xacro:include filename="$(find akros2_description)/urdf/akros2_mecanum/akros2_mecanum.common.xacro"/>
-<xacro:include filename="$(find akros2_description)/urdf/akros2_mecanum/akros2_mecanum.control.xacro"/>
-<xacro:include filename="$(find akros2_description)/urdf/akros2_mecanum/akros2_mecanum.gazebo.xacro"/>
+<xacro:include filename="$(find akros2_description)/urdf/akros2_mecanum/robot.common.xacro"/>
+<xacro:include filename="$(find akros2_description)/urdf/akros2_mecanum/robot.control.xacro"/>
+<xacro:include filename="$(find akros2_description)/urdf/akros2_mecanum/robot.gazebo.xacro"/>
 <xacro:arg name="mesh_path" default="package://akros2_description/meshes/akros2_mecanum/" /> <!-- HTTPS URL also works here -->
 <xacro:arg name="unity" default="false" />
@@ -11,4 +11,6 @@
 </xacro:if>
 <!-- **** LINKS **** -->
+<!-- BASE_FOOTPRINT -->
+<link name="base_footprint"/>
 <!-- BASE_LINK -->
 <link name="base_link">
@@ -35,6 +37,4 @@
   </inertial>
 </link>
-<!-- BASE_FOOTPRINT -->
-<link name="base_footprint"/>
 <!-- NAV_LINK -->
 <link name="nav_link">
@@ -165,4 +165,10 @@
 </link>
 <!-- **** JOINTS **** -->
+<!-- BASE_LINK TO BASE_FOOTPRINT -->
+<joint name="footprint_base_fixed" type="fixed">
+  <parent link="base_footprint"/>
+  <child link="base_link"/>
+  <origin xyz="0 0 ${footprint_base_offset_z}"/>
+</joint>
 <!-- BASE_LINK_INERTIAL TO BASE_LINK -->
 <joint name="base_inertial_fixed" type="fixed">
@@ -170,10 +176,4 @@
   <child link="base_link_inertial"/>
   <origin xyz="0 0 0"/>
-</joint>
-<!-- BASE_FOOTPRINT TO BASE_LINK -->
-<joint name="base_footprint_fixed" type="fixed">
-  <parent link="base_link"/>
-  <child link="base_footprint"/>
-  <origin xyz="0 0 ${base_footprint_offset_z}"/>
 </joint>
 <!-- NAV_LINK TO BASE_LINK -->

File: urdf/akros2_omni/robot.common.xacro (robot description, xacro)
@@ -1,4 +1,4 @@
 <?xml version="1.0" encoding="utf-8"?>
-<robot name="mecanum_common" xmlns:xacro="http://ros.org/wiki/xacro">
+<robot name="omni_common" xmlns:xacro="http://ros.org/wiki/xacro">
 <!-- All values below are based on CAD model (Fusion 360). 2mm added on each side (4mm total) for length and width (but not height) as padding. -->
 <xacro:property name="pi_by_two" value="1.5707963" />
@@ -23,5 +23,5 @@
 <xacro:property name="wheel_mass" value="0.075" /> <!-- Guesstimate, needs to be measured -->
 <xacro:property name="wheel_thickness" value="0.034" /> <!-- Actual thickness = 0.034, CAD thickness = 0.0315 -->
-<xacro:property name="base_footprint_offset_z" value="-0.017877" /> <!-- Actual offset = -0.017877, CAD offset = -0.015377 -->
+<xacro:property name="footprint_base_offset_z" value="0.017877" /> <!-- Actual offset = 0.017877, CAD offset = 0.015377 -->
 <xacro:property name="nav_laser_offset_x" value="0.0632" />
 <xacro:property name="laser_frame_offset_z" value="0.0255" />

File: urdf/akros2_omni/robot.control.xacro (robot description, xacro)
@@ -12,5 +12,5 @@
   </actuator>
 </transmission>
-<!-- WHEEL_L (BACK) TRANSMISSION -->
+<!-- WHEEL_L TRANSMISSION -->
 <transmission name="trans_l">
   <type>transmission_interface/SimpleTransmission</type>
@@ -23,5 +23,5 @@
   </actuator>
 </transmission>
-<!-- WHEEL_R (BACK) TRANSMISSION -->
+<!-- WHEEL_R TRANSMISSION -->
 <transmission name="trans_r">
   <type>transmission_interface/SimpleTransmission</type>

File: urdf/akros2_omni/robot.gazebo.xacro (robot description, xacro)
@@ -1,4 +1,4 @@
 <?xml version="1.0" encoding="utf-8"?>
-<robot name="mecanum_gazebo" xmlns:xacro="http://ros.org/wiki/xacro">
+<robot name="omni_gazebo" xmlns:xacro="http://ros.org/wiki/xacro">
 <gazebo reference="base_link">
   <material>Gazebo/Grey</material>
@@ -10,14 +10,11 @@
   <material>Gazebo/FlatBlack</material>
 </gazebo>
-<gazebo reference="wheel_lf">
+<gazebo reference="wheel_f">
   <material>Gazebo/DarkGrey</material>
 </gazebo>
-<gazebo reference="wheel_lb">
+<gazebo reference="wheel_l">
   <material>Gazebo/DarkGrey</material>
 </gazebo>
-<gazebo reference="wheel_rf">
-  <material>Gazebo/DarkGrey</material>
-</gazebo>
-<gazebo reference="wheel_rb">
+<gazebo reference="wheel_r">
   <material>Gazebo/DarkGrey</material>
 </gazebo>
@@ -87,5 +84,5 @@
     <odometryFrame>odom</odometryFrame>
     <odometryRate>100.0</odometryRate>
-    <robotBaseFrame>base_link</robotBaseFrame>
+    <robotBaseFrame>base_footprint</robotBaseFrame>
     <publishTF>false</publishTF>
   </plugin>

File: urdf/akros2_omni/robot.urdf (robot description, URDF)
Before this commit: robot akros2_omni, 11 links, 10 joints
Links:
- link base_link: geometry collision box size=0.21038 0.1585 0.099; visual mesh filename=package://akros2_description/meshes/akros2_mecanum/base_mod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
- link laser_link: geometry collision box size=0.042 0.0421 0.033; visual mesh filename=package://akros2_description/meshes/akros2_mecanum/ld06.dae
- link nav_link: geometry collision box size=0.2044 0.1585 0.03065; visual mesh filename=package://akros2_description/meshes/akros2_mecanum/navigati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
- link wheel_f: geometry collision cylinder length=0.034 radius=0.0385; visual mesh filename=package://akros2_description/meshes/akros2_mecanum/wheel_f.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
- link wheel_l: geometry collision cylinder length=0.034 radius=0.0385; visual mesh filename=package://akros2_description/meshes/akros2_mecanum/wheel_l.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
- link wheel_r: geometry collision cylinder length=0.034 radius=0.0385; visual mesh filename=package://akros2_description/meshes/akros2_mecanum/wheel_r.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
Joints:
- removed joint base_footprint_fixed
- added joint footprint_base_fixed: type fixed, parent base_footprint, child base_link, origin xyz=0 0 0.017877
- joint imu_base_fixed: origin xyz=0 0 0 -> xyz=0.0562 0 0.094
- joint joint_f: origin xyz=0.0495 0.078 0.021 rpy=0 0 0 -> xyz=0.0495 0.0854225 0.021 rpy=0 0 0
- joint joint_l: origin xyz=-0.0495 0.078 0.021 rpy=0 0 0 -> xyz=-0.0495 0.0854225 0.021 rpy=0 0 0
- joint joint_r: origin xyz=0.0495 -0.078 0.021 rpy=0 0 0 -> xyz=0.0495 -0.0854225 0.021 rpy=0 0 0

File: urdf/akros2_omni/robot.urdf.xacro (robot description, xacro)
@@ -1,7 +1,7 @@
 <?xml version="1.0" encoding="utf-8"?>
 <robot name="akros2_omni" xmlns:xacro="http://ros.org/wiki/xacro">
-<xacro:include filename="$(find akros2_description)/urdf/akros2_omni/akros2_omni.common.xacro"/>
-<xacro:include filename="$(find akros2_description)/urdf/akros2_omni/akros2_omni.control.xacro"/>
-<xacro:include filename="$(find akros2_description)/urdf/akros2_omni/akros2_omni.gazebo.xacro"/>
+<xacro:include filename="$(find akros2_description)/urdf/akros2_omni/robot.common.xacro"/>
+<xacro:include filename="$(find akros2_description)/urdf/akros2_omni/robot.control.xacro"/>
+<xacro:include filename="$(find akros2_description)/urdf/akros2_omni/robot.gazebo.xacro"/>
 <xacro:arg name="mesh_path" default="package://akros2_description/meshes/akros2_omni/" /> <!-- HTTPS URL also works here -->
 <xacro:arg name="unity" default="false" />
@@ -11,4 +11,6 @@
 </xacro:if>
 <!-- **** LINKS **** -->
+<!-- BASE_FOOTPRINT -->
+<link name="base_footprint"/>
 <!-- BASE_LINK -->
 <link name="base_link">
@@ -18,8 +20,8 @@
       <mesh filename="${mesh_path}base_module.dae" />
     </geometry>
-   <material name="White"/>
-  </visual>
-  <collision>
-    <origin xyz="${base_offset_x} 0 ${base_height/2}" rpy="0 0 0" /> <!-- If needed: offset from ground = 0.0278 -->
+   <material name="BaseLinkColor"/>
+  </visual>
+  <collision>
+    <origin xyz="${base_offset_x/2} 0 ${base_height/2}" rpy="0 0 0" />
     <geometry>
       <box size="${base_length} ${base_width} ${base_height}"/>
@@ -35,6 +37,4 @@
   </inertial>
 </link>
-<!-- BASE_FOOTPRINT -->
-<link name="base_footprint"/>
 <!-- NAV_LINK -->
 <link name="nav_link">
@@ -44,12 +44,12 @@
   </inertial>
   <visual>
-    <origin xyz="0 0 -0.099" rpy="0 0 0" />
+    <origin xyz="0 0 ${nav_offset_z}" rpy="0 0 0" />
     <geometry>
       <mesh filename="${mesh_path}navigation_module.dae" />
     </geometry>
-    <material name="DarkGrey"/>
-  </visual>
-  <collision>
-    <origin xyz="0 0 ${nav_height/2}" rpy="0 0 0" /> <!-- If needed: offset from base_link = -0.099 -->
+    <material name="WheelsNavColor"/>
+  </visual>
+  <collision>
+    <origin xyz="0 0 ${nav_height/2}" rpy="0 0 0" />
     <geometry>
       <box size="${nav_length} ${nav_width} ${nav_height}"/>
@@ -69,5 +69,5 @@
       <mesh filename="${mesh_path}ld06.dae" />
     </geometry>
-    <material name="FlatBlack"/>
+    <material name="LaserColor"/>
   </visual>
   <collision>
@@ -88,5 +88,5 @@
   <inertial>
     <mass value="${wheel_mass}"/>
-    <xacro:cylinder_inertia m="${wheel_mass}" r="${wheel_radius}" h="${wheel_height}"/>
+    <xacro:cylinder_inertia m="${wheel_mass}" r="${wheel_radius}" h="${wheel_thickness}"/>
   </inertial>
   <visual>
@@ -95,18 +95,18 @@
       <mesh filename="${mesh_path}wheel_f.dae" />
     </geometry>
-    <material name="FlatBlack"/>
-  </visual>
-  <collision>
-    <origin xyz="0 ${wheel_height/2} 0" rpy="${pi_by_two} 0 0" /><!-- If needed: offset from joint = 0.01 -->
-    <geometry>
-      <cylinder length="${wheel_height}" radius="${wheel_radius}"/>
-    </geometry>
-  </collision>
-</link>
-<!-- WHEEL LEFT (BACK) -->
+    <material name="WheelsNavColor"/>
+  </visual>
+  <collision>
+    <origin xyz="0 ${wheel_thickness/2} 0" rpy="${pi_by_two} 0 0" />
+    <geometry>
+      <cylinder length="${wheel_thickness}" radius="${wheel_radius}"/>
+    </geometry>
+  </collision>
+</link>
+<!-- WHEEL LEFT -->
 <link name="wheel_l">
   <inertial>
     <mass value="${wheel_mass}"/>
-    <xacro:cylinder_inertia m="${wheel_mass}" r="${wheel_radius}" h="${wheel_height}"/>
+    <xacro:cylinder_inertia m="${wheel_mass}" r="${wheel_radius}" h="${wheel_thickness}"/>
   </inertial>
   <visual>
@@ -115,18 +115,18 @@
       <mesh filename="${mesh_path}wheel_l.dae" />
     </geometry>
-    <material name="FlatBlack"/>
-  </visual>
-  <collision>
-    <origin xyz="0 ${wheel_height/2} 0" rpy="${pi_by_two} 0 0" /><!-- If needed: offset from joint = 0.01 -->
-    <geometry>
-      <cylinder length="${wheel_height}" radius="${wheel_radius}"/>
-    </geometry>
-  </collision>
-</link>
-<!-- WHEEL RIGHT (BACK) -->
+    <material name="WheelsNavColor"/>
+  </visual>
+  <collision>
+    <origin xyz="0 ${wheel_thickness/2} 0" rpy="${pi_by_two} 0 0" />
+    <geometry>
+      <cylinder length="${wheel_thickness}" radius="${wheel_radius}"/>
+    </geometry>
+  </collision>
+</link>
+<!-- WHEEL RIGHT FRONT -->
 <link name="wheel_r">
   <inertial>
     <mass value="${wheel_mass}"/>
-    <xacro:cylinder_inertia m="${wheel_mass}" r="${wheel_radius}" h="${wheel_height}"/>
+    <xacro:cylinder_inertia m="${wheel_mass}" r="${wheel_radius}" h="${wheel_thickness}"/>
   </inertial>
   <visual>
@@ -135,24 +135,24 @@
       <mesh filename="${mesh_path}wheel_r.dae" />
     </geometry>
-    <material name="FlatBlack"/>
-  </visual>
-  <collision>
-    <origin xyz="0 ${-1*(wheel_height/2)} 0" rpy="${pi_by_two} 0 0" /><!-- If needed: offset from joint = 0.01 -->
-    <geometry>
-      <cylinder length="${wheel_height}" radius="${wheel_radius}"/>
+    <material name="WheelsNavColor"/>
+  </visual>
+  <collision>
+    <origin xyz="0 ${-1*(wheel_thickness/2)} 0" rpy="${pi_by_two} 0 0" />
+    <geometry>
+      <cylinder length="${wheel_thickness}" radius="${wheel_radius}"/>
     </geometry>
   </collision>
 </link>
 <!-- **** JOINTS **** -->
+<!-- BASE_LINK TO BASE_FOOTPRINT -->
+<joint name="footprint_base_fixed" type="fixed">
+  <parent link="base_footprint"/>
+  <child link="base_link"/>
+  <origin xyz="0 0 ${footprint_base_offset_z}"/>
+</joint>
 <!-- BASE_LINK_INERTIAL TO BASE_LINK -->
 <joint name="base_inertial_fixed" type="fixed">
   <parent link="base_link"/>
   <child link="base_link_inertial"/>
-  <origin xyz="0 0 0"/>
-</joint>
-<!-- BASE_FOOTPRINT TO BASE_LINK -->
-<joint name="base_footprint_fixed" type="fixed">
-  <parent link="base_link"/>
-  <child link="base_footprint"/>
   <origin xyz="0 0 0"/>
 </joint>
@@ -180,5 +180,5 @@
   <parent link="base_link"/>
   <child link="imu_link"/>
-  <origin xyz="0 0 0"/>
+  <origin xyz="${imu_offset_x} 0 ${imu_offset_z}"/>
 </joint>
 <!-- IMU_FRAME TO IMU_LINK -->
@@ -195,5 +195,5 @@
   <axis xyz="0 1 0" />
 </joint>
-<!-- WHEEL_L (BACK) TO BASE_LINK -->
+<!-- WHEEL_L TO BASE_LINK -->
 <joint name="joint_l" type="continuous">
   <parent link="base_link" />
@@ -202,5 +202,5 @@
   <axis xyz="0 1 0" />
 </joint>
-<!-- WHEEL_R (BACK) TO BASE_LINK -->
+<!-- WHEEL_R TO BASE_LINK -->
 <joint name="joint_r" type="continuous">
   <parent link="base_link" />

Commit message: update imu_frame to imu_link

File: urdf/akros2_mecanum/robot.gazebo.xacro (robot description, xacro)
@@ -56,6 +56,6 @@
   <plugin name="imu_plugin" filename="libgazebo_ros_imu.so">
     <alwaysOn>true</alwaysOn>
-    <bodyName>imu_frame</bodyName>
-    <frameName>imu_frame</frameName>
+    <bodyName>imu_link</bodyName>
+    <frameName>imu_link</frameName>
     <topicName>imu</topicName>
     <serviceName>imu_service</serviceName>

File: urdf/akros2_mecanum/robot.urdf (robot description, URDF)
Before this commit: robot akros2_mecanum, 11 links, 10 joints
Links:
- removed link imu_frame
- added link imu_link
Joints:
- joint imu_base_fixed: child imu_frame -> imu_link

File: urdf/akros2_mecanum/robot.urdf.xacro (robot description, xacro)
@@ -81,5 +81,5 @@
 <link name="laser_frame"/>
 <!-- MPU9250 IMU_LINK -->
-<link name="imu_frame"/>
+<link name="imu_link"/>
 <!-- WHEEL LEFT FRONT -->
 <link name="wheel_lf">
@@ -197,5 +197,5 @@
 <joint name="imu_base_fixed" type="fixed">
   <parent link="base_link"/>
-  <child link="imu_frame"/>
+  <child link="imu_link"/>
   <origin xyz="${imu_offset_x} 0 ${imu_offset_z}"/>
 </joint>

File: urdf/akros2_omni/robot.gazebo.xacro (robot description, xacro)
@@ -53,6 +53,6 @@
   <plugin name="imu_plugin" filename="libgazebo_ros_imu.so">
     <alwaysOn>true</alwaysOn>
-    <bodyName>imu_frame</bodyName>
-    <frameName>imu_frame</frameName>
+    <bodyName>imu_link</bodyName>
+    <frameName>imu_link</frameName>
     <topicName>imu</topicName>
     <serviceName>imu_service</serviceName>

File: urdf/akros2_omni/robot.urdf (robot description, URDF)
Before this commit: robot akros2_omni, 11 links, 10 joints
Links:
- removed link imu_frame
Joints:
- removed joint imu_frame_fixed

File: urdf/akros2_omni/robot.urdf.xacro (robot description, xacro)
@@ -82,6 +82,4 @@
 <!-- MPU9250 IMU_LINK -->
 <link name="imu_link"/>
-<!-- IMU_FRAME -->
-<link name="imu_frame"/>
 <!-- WHEEL FRONT -->
 <link name="wheel_f">
@@ -182,10 +180,4 @@
   <origin xyz="${imu_offset_x} 0 ${imu_offset_z}"/>
 </joint>
-<!-- IMU_FRAME TO IMU_LINK -->
-<joint name="imu_frame_fixed" type="fixed">
-  <parent link="imu_link"/>
-  <child link="imu_frame"/>
-  <origin xyz="0 0 0"/>
-</joint>
 <!-- WHEEL_F TO BASE_LINK -->
 <joint name="joint_f" type="continuous">
