Commit message: add camera module

File: urdf/akros2_mecanum/robot.common.xacro (robot description, xacro)
@@ -19,5 +19,9 @@
 <xacro:property name="laser_length" value="0.042" /> <!-- Actual length without padding = 0.038 -->
 <xacro:property name="laser_width" value="0.0421" /> <!-- Actual width without padding = 0.0381 -->
-<xacro:property name="laser_height" value="0.033" />
+<xacro:property name="laser_height" value="0.033"/>
+<xacro:property name="cam_mass" value="0.025" />
+<xacro:property name="cam_length" value="0.0161" /> <!-- Actual length without padding = 0.0121 -->
+<xacro:property name="cam_width" value="0.0730" /> <!-- Actual width without padding = 0.0690 -->
+<xacro:property name="cam_height" value="0.01" />
 <xacro:property name="wheel_radius" value="0.0385" /> <!-- Actual radius = 0.0385, CAD radius = 0.036 -->
 <xacro:property name="wheel_mass" value="0.075" /> <!-- Guesstimate, needs to be measured -->
@@ -26,4 +30,7 @@
 <xacro:property name="nav_laser_offset_x" value="0.0632" />
 <xacro:property name="laser_frame_offset_z" value="0.0255" />
+<xacro:property name="nav_cam_offset_x" value="0.0877" />
+<xacro:property name="nav_cam_offset_z" value="0.01525" />
+<xacro:property name="cam_frame_offset_x" value="0.0065" />
 <xacro:property name="joint_offset_x" value="0.0495" />
 <xacro:property name="joint_offset_y" value="0.0854225" />
@@ -44,5 +51,5 @@
             izz="${2*m*r*r/5}" />
 </xacro:macro>
-<material name="LaserColor">
+<material name="SensorColor">
     <color rgba="0.2 0.2 0.2 1"/>
 </material>

File: urdf/akros2_mecanum/robot.gazebo.xacro (robot description, xacro)
@@ -8,4 +8,7 @@
 </gazebo>
 <gazebo reference="laser_link">
+  <material>Gazebo/FlatBlack</material>
+</gazebo>
+<gazebo reference="cam_link">
   <material>Gazebo/FlatBlack</material>
 </gazebo>

File: urdf/akros2_mecanum/robot.urdf (robot description, URDF)
Before this commit: robot akros2_mecanum, 11 links, 10 joints
Links:
- added link cam_frame
- added link cam_link, mass 0.025; collision box size=0.0161 0.0421 0.033; visual mesh filename=package://akros2_description/meshes/akros2_mecanum/cam_modu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
Joints:
- added joint cam_frame_fixed: type fixed, parent cam_link, child cam_frame, origin xyz=0.0065 0 0 rpy=-1.5707963 0 -1.5707963
- added joint nav_cam_fixed: type fixed, parent nav_link, child cam_link, origin xyz=0.0877 0 0.01525
- joint nav_laser_fixed: origin xyz=0.0632 0 0.0155 -> xyz=0.0632 0 0.015325

File: urdf/akros2_mecanum/robot.urdf.xacro (robot description, xacro)
@@ -69,5 +69,5 @@
       <mesh filename="${mesh_path}ld06.dae" />
     </geometry>
-    <material name="LaserColor"/>
+    <material name="SensorColor"/>
   </visual>
   <collision>
@@ -80,4 +80,27 @@
 <!-- LASER_FRAME -->
 <link name="laser_frame"/>
+<!-- USB CAMERA MODULE CAM_LINK -->
+<link name="cam_link">
+  <inertial>
+    <origin xyz="0 0 0" rpy="0 0 0" />
+    <mass value="${cam_mass}" />
+    <xacro:box_inertia m="${cam_mass}" x="${cam_length}" y="${cam_width}" z="${cam_height}"/>
+  </inertial>
+  <visual>
+    <origin xyz="0 0 0" rpy="0 0 0" />
+    <geometry>
+      <mesh filename="${mesh_path}cam_module.dae" />
+    </geometry>
+    <material name="SensorColor"/>
+  </visual>
+  <collision>
+    <origin xyz="${cam_length/2} 0 0" rpy="0 0 0" />
+    <geometry>
+      <box size="${cam_length} ${laser_width} ${laser_height}"/>
+    </geometry>
+  </collision>
+</link>
+<!-- USB CAMERA OPTICAL FRAME CAM_FRAME -->
+<link name="cam_frame"/>
 <!-- MPU9250 IMU_LINK -->
 <link name="imu_link"/>
@@ -194,4 +217,16 @@
   <origin xyz="0 0 ${laser_frame_offset_z}"/>
 </joint>
+<!-- CAM_LINK TO NAV_LINK -->
+<joint name="nav_cam_fixed" type="fixed">
+  <parent link="nav_link"/>
+  <child link="cam_link"/>
+  <origin xyz="${nav_cam_offset_x} 0 ${nav_cam_offset_z}"/>
+</joint>
+<!-- CAM_FRAME TO CAM_LINK -->
+<joint name="cam_frame_fixed" type="fixed">
+  <parent link="cam_link"/>
+  <child link="cam_frame"/>
+  <origin xyz="${cam_frame_offset_x} 0 0" rpy="${minus_pi_by_two} 0 ${minus_pi_by_two}"/>
+</joint>
 <!-- IMU_LINK TO BASE_LINK -->
 <joint name="imu_base_fixed" type="fixed">

Commit message: added omni URDF - WIP

File: urdf/akros2_mecanum/robot.common.xacro (robot description, xacro)
@@ -3,5 +3,4 @@
 <!-- All values below are based on CAD model (Fusion 360). 2mm added on each side (4mm total) for length and width (but not height) as padding. -->
 <xacro:property name="pi_by_two" value="1.5707963" />
-<xacro:property name="minus_pi_by_two" value="-1.5707963" />
 <xacro:property name="base_mass" value="2.0" /> <!-- Guesstimate, needs to be measured -->
 <xacro:property name="base_length" value="0.21038" /> <!-- Actual length without padding = 0.20638. Change to 0.21038 to include screw heads in collision (without padding). -->

File: urdf/akros2_mecanum/robot.urdf.xacro (robot description, xacro)
@@ -65,5 +65,5 @@
   </inertial>
   <visual>
-    <origin xyz="0 0 0" rpy="0 0 ${minus_pi_by_two}" />
+    <origin xyz="0 0 0" rpy="0 0 ${-1*pi_by_two}" />
     <geometry>
       <mesh filename="${mesh_path}ld06.dae" />
@@ -72,5 +72,5 @@
   </visual>
   <collision>
-    <origin xyz="0 0 ${laser_height/2}" rpy="0 0 ${minus_pi_by_two}" />
+    <origin xyz="0 0 ${laser_height/2}" rpy="0 0 ${-1*pi_by_two}" />
     <geometry>
       <box size="${laser_length} ${laser_width} ${laser_height}"/>
@@ -227,5 +227,5 @@
   <parent link="cam_link"/>
   <child link="cam_frame"/>
-  <origin xyz="${cam_frame_offset_x} 0 0" rpy="${minus_pi_by_two} 0 ${minus_pi_by_two}"/>
+  <origin xyz="${cam_frame_offset_x} 0 0" rpy="${-1*pi_by_two} 0 ${-1*pi_by_two}"/>
 </joint>
 <!-- IMU_LINK TO BASE_LINK -->

File: urdf/akros2_omni/robot.common.xacro (robot description, xacro)
@@ -3,30 +3,25 @@
 <!-- All values below are based on CAD model (Fusion 360). 2mm added on each side (4mm total) for length and width (but not height) as padding. -->
 <xacro:property name="pi_by_two" value="1.5707963" />
-<xacro:property name="minus_pi_by_two" value="-1.5707963" />
+<xacro:property name="pi_by_three" value="1.0471975"/>
 <xacro:property name="base_mass" value="2.0" /> <!-- Guesstimate, needs to be measured -->
-<xacro:property name="base_length" value="0.21038" /> <!-- Actual length without padding = 0.20638. Change to 0.21038 to include screw heads in collision (without padding). -->
-<xacro:property name="base_width" value="0.1585" /> <!-- Actual width without padding = 0.1545 without screw heads. Change to 0.2 to include motor shafts and emergency button (without padding)-->
-<xacro:property name="base_height" value="0.099" />
-<xacro:property name="base_offset_x" value="0.006" />
-<xacro:property name="nav_offset_z" value="-0.099" />
-<xacro:property name="nav_mass" value="0.5" /> <!-- Guesstimate, needs to be measured -->
-<xacro:property name="nav_length" value="0.2044" /> <!-- Actual length without padding = 0.2004 -->
-<xacro:property name="nav_width" value="0.1585" /> <!-- Actual width without padding = 0.1545-->
-<xacro:property name="nav_height" value="0.03065" />
-<xacro:property name="imu_offset_x" value="0.0562" />
-<xacro:property name="imu_offset_z" value="0.094" />
+<xacro:property name="base_height" value="0.1673" />
+<xacro:property name="base_radius" value="0.105" /> <!-- Distance from the motor shaft to the vertical axis -->
+<xacro:property name="imu_offset_z" value="0.063003" />
 <xacro:property name="laser_mass" value="0.12" />
-<xacro:property name="laser_length" value="0.042" /> <!-- Actual length without padding = 0.038 -->
-<xacro:property name="laser_width" value="0.0421" /> <!-- Actual width without padding = 0.0381 -->
+<xacro:property name="laser_length" value="0.038" />
+<xacro:property name="laser_width" value="0.0381" />
 <xacro:property name="laser_height" value="0.033" />
-<xacro:property name="wheel_radius" value="0.0385" /> <!-- Actual radius = 0.0385, CAD radius = 0.036 -->
+<xacro:property name="wheel_radius" value="0.029" />
 <xacro:property name="wheel_mass" value="0.075" /> <!-- Guesstimate, needs to be measured -->
-<xacro:property name="wheel_thickness" value="0.034" /> <!-- Actual thickness = 0.034, CAD thickness = 0.0315 -->
-<xacro:property name="footprint_base_offset_z" value="0.017877" /> <!-- Actual offset = 0.017877, CAD offset = 0.015377 -->
-<xacro:property name="nav_laser_offset_x" value="0.0632" />
+<xacro:property name="wheel_thickness" value="0.026" />
+<xacro:property name="base_center_offset_z" value="0.0170" />
+<xacro:property name="footprint_base_offset_z" value="0.085597" /> <!-- CAD offset, Actual offset ~= 0.083597 -->
+<xacro:property name="base_laser_offset_x" value="0.034435" />
+<xacro:property name="base_laser_offset_z" value="0.076503" />
 <xacro:property name="laser_frame_offset_z" value="0.0255" />
-<xacro:property name="joint_offset_x" value="0.0495" />
-<xacro:property name="joint_offset_y" value="0.0854225" />
-<xacro:property name="joint_offset_z" value="0.021" />
+<xacro:property name="joint_f_offset_x" value="0.10683" />
+<xacro:property name="joint_lr_offset_x" value="-0.053415" />
+<xacro:property name="joint_lr_offset_y" value="0.092518" />
+<xacro:property name="joint_offset_z" value="-0.056597" />
 <xacro:macro name="cylinder_inertia" params="m r h">
   <inertia  ixx="${m*(3*r*r+h*h)/12}" ixy = "0" ixz = "0"

File: urdf/akros2_omni/robot.gazebo.xacro (robot description, xacro)
@@ -3,7 +3,4 @@
 <gazebo reference="base_link">
   <material>Gazebo/Grey</material>
-</gazebo>
-<gazebo reference="nav_link">
-  <material>Gazebo/DarkGrey</material>
 </gazebo>
 <gazebo reference="laser_link">

File: urdf/akros2_omni/robot.urdf.xacro (robot description, xacro)
@@ -20,10 +20,10 @@
       <mesh filename="${mesh_path}base_module.dae" />
     </geometry>
-   <material name="BaseLinkColor"/>
+    <material name="BaseLinkColor"/>
   </visual>
   <collision>
-    <origin xyz="${base_offset_x/2} 0 ${base_height/2}" rpy="0 0 0" />
+    <origin xyz="0 0 ${base_center_offset_z}" rpy="0 0 0" />
     <geometry>
-      <box size="${base_length} ${base_width} ${base_height}"/>
+      <cylinder length="${base_height}" radius="${base_radius}"/>
     </geometry>
   </collision>
@@ -34,26 +34,6 @@
     <origin xyz="0 0 0" rpy="0 0 0" />
     <mass value="${base_mass}"/>
-    <xacro:box_inertia m="${base_mass}" x="${base_length}" y="${base_width}" z="${base_height}"/>
+    <xacro:cylinder_inertia m="${base_mass}" r="${base_radius}" h="${base_height}"/>
   </inertial>
-</link>
-<!-- NAV_LINK -->
-<link name="nav_link">
-  <inertial>
-    <mass value="${nav_mass}" />
-    <xacro:box_inertia m="${nav_mass}" x="${nav_length}" y="${nav_width}" z="${nav_height}"/>
-  </inertial>
-  <visual>
-    <origin xyz="0 0 ${nav_offset_z}" rpy="0 0 0" />
-    <geometry>
-      <mesh filename="${mesh_path}navigation_module.dae" />
-    </geometry>
-    <material name="WheelsNavColor"/>
-  </visual>
-  <collision>
-    <origin xyz="0 0 ${nav_height/2}" rpy="0 0 0" />
-    <geometry>
-      <box size="${nav_length} ${nav_width} ${nav_height}"/>
-    </geometry>
-  </collision>
 </link>
 <!-- LD06 LASER_LINK -->
@@ -65,5 +45,5 @@
   </inertial>
   <visual>
-    <origin xyz="0 0 0" rpy="0 0 ${minus_pi_by_two}" />
+    <origin xyz="0 0 0" rpy="0 0 ${-1*pi_by_two}" />
     <geometry>
       <mesh filename="${mesh_path}ld06.dae" />
@@ -72,5 +52,5 @@
   </visual>
   <collision>
-    <origin xyz="0 0 ${laser_height/2}" rpy="0 0 ${minus_pi_by_two}" />
+    <origin xyz="0 0 ${laser_height/2}" rpy="0 0 ${-1*pi_by_two}" />
     <geometry>
       <box size="${laser_length} ${laser_width} ${laser_height}"/>
@@ -91,10 +71,10 @@
     <origin xyz="0 0 0" rpy="0 0 0" />
     <geometry>
-      <mesh filename="${mesh_path}wheel_f.dae" />
+      <mesh filename="${mesh_path}omniwheel.dae" />
     </geometry>
     <material name="WheelsNavColor"/>
   </visual>
   <collision>
-    <origin xyz="0 ${wheel_thickness/2} 0" rpy="${pi_by_two} 0 0" />
+    <origin xyz="${wheel_thickness/2} 0 0" rpy="0 ${pi_by_two} 0" />
     <geometry>
       <cylinder length="${wheel_thickness}" radius="${wheel_radius}"/>
@@ -111,10 +91,10 @@
     <origin xyz="0 0 0" rpy="0 0 0" />
     <geometry>
-      <mesh filename="${mesh_path}wheel_l.dae" />
+      <mesh filename="${mesh_path}omniwheel.dae" />
     </geometry>
     <material name="WheelsNavColor"/>
   </visual>
   <collision>
-    <origin xyz="0 ${wheel_thickness/2} 0" rpy="${pi_by_two} 0 0" />
+    <origin xyz="${wheel_thickness/2} 0 0" rpy="0 ${pi_by_two} 0" />
     <geometry>
       <cylinder length="${wheel_thickness}" radius="${wheel_radius}"/>
@@ -122,5 +102,5 @@
   </collision>
 </link>
-<!-- WHEEL RIGHT FRONT -->
+<!-- WHEEL RIGHT -->
 <link name="wheel_r">
   <inertial>
@@ -131,10 +111,10 @@
     <origin xyz="0 0 0" rpy="0 0 0" />
     <geometry>
-      <mesh filename="${mesh_path}wheel_r.dae" />
+      <mesh filename="${mesh_path}omniwheel.dae" />
     </geometry>
     <material name="WheelsNavColor"/>
   </visual>
   <collision>
-    <origin xyz="0 ${-1*(wheel_thickness/2)} 0" rpy="${pi_by_two} 0 0" />
+    <origin xyz="${wheel_thickness/2} 0 0" rpy="0 ${pi_by_two} 0" />
     <geometry>
       <cylinder length="${wheel_thickness}" radius="${wheel_radius}"/>
@@ -155,16 +135,9 @@
   <origin xyz="0 0 0"/>
 </joint>
-<!-- NAV_LINK TO BASE_LINK -->
-<joint name="base_nav_fixed" type="fixed">
+<!-- LASER_LINK TO BASE_LINK -->
+<joint name="base_laser_fixed" type="fixed">
   <parent link="base_link"/>
-  <child link="nav_link"/>
-  <origin xyz="0 0 ${base_height}"/>
-  <axis xyz="0 0 0"/>
-</joint>
-<!-- LASER_LINK TO NAV_LINK -->
-<joint name="nav_laser_fixed" type="fixed">
-  <parent link="nav_link"/>
   <child link="laser_link"/>
-  <origin xyz="${nav_laser_offset_x} 0 ${nav_height/2}"/>
+  <origin xyz="${base_laser_offset_x} 0 ${base_laser_offset_z}"/>
 </joint>
 <!-- LASER_FRAME TO LASER_LINK -->
@@ -178,5 +151,5 @@
   <parent link="base_link"/>
   <child link="imu_link"/>
-  <origin xyz="${imu_offset_x} 0 ${imu_offset_z}"/>
+  <origin xyz="0 0 ${imu_offset_z}"/>
 </joint>
 <!-- WHEEL_F TO BASE_LINK -->
@@ -184,6 +157,6 @@
   <parent link="base_link" />
   <child link="wheel_f" />
-  <origin xyz="${joint_offset_x} ${joint_offset_y} ${joint_offset_z}" rpy="0 0 0" />
-  <axis xyz="0 1 0" />
+  <origin xyz="${joint_f_offset_x} 0 ${joint_offset_z}" rpy="0 0 0" />
+  <axis xyz="1 0 0" />
 </joint>
 <!-- WHEEL_L TO BASE_LINK -->
@@ -191,6 +164,6 @@
   <parent link="base_link" />
   <child link="wheel_l" />
-  <origin xyz="${-1*joint_offset_x} ${joint_offset_y} ${joint_offset_z}" rpy="0 0 0" />
-  <axis xyz="0 1 0" />
+  <origin xyz="${joint_lr_offset_x} ${joint_lr_offset_y} ${joint_offset_z}" rpy="0 0 ${2*pi_by_three}" />
+  <axis xyz="1 0 0" />
 </joint>
 <!-- WHEEL_R TO BASE_LINK -->
@@ -198,6 +171,6 @@
   <parent link="base_link" />
   <child link="wheel_r" />
-  <origin xyz="${joint_offset_x} ${-1*joint_offset_y} ${joint_offset_z}" rpy="0 0 0" />
-  <axis xyz="0 1 0" />
+  <origin xyz="${joint_lr_offset_x} ${-1*joint_lr_offset_y} ${joint_offset_z}" rpy="0 0 ${-2*pi_by_three}" />
+  <axis xyz="1 0 0" />
 </joint>
 </robot>

Commit message: update

File: urdf/akros2_mecanum/robot.common.xacro (robot description, xacro)
@@ -1,5 +1,5 @@
 <?xml version="1.0" encoding="utf-8"?>
 <robot name="mecanum_common" xmlns:xacro="http://ros.org/wiki/xacro">
-<!-- All values below are based on CAD model (Fusion 360). 2mm added on each side (4mm total) for length and width (but not height) as padding. -->
+<!-- All values below are based on the CAD model (Fusion 360). 2mm added on each side (4mm total) for length and width (but not height) as padding. -->
 <xacro:property name="pi_by_two" value="1.5707963" />
 <xacro:property name="base_mass" value="2.0" /> <!-- Guesstimate, needs to be measured -->

File: urdf/akros2_omni/robot.common.xacro (robot description, xacro)
@@ -1,9 +1,9 @@
 <?xml version="1.0" encoding="utf-8"?>
 <robot name="omni_common" xmlns:xacro="http://ros.org/wiki/xacro">
-<!-- All values below are based on CAD model (Fusion 360). 2mm added on each side (4mm total) for length and width (but not height) as padding. -->
+<!-- All values below are based on the CAD model (Fusion 360) -->
 <xacro:property name="pi_by_two" value="1.5707963" />
 <xacro:property name="pi_by_three" value="1.0471975"/>
 <xacro:property name="base_mass" value="2.0" /> <!-- Guesstimate, needs to be measured -->
-<xacro:property name="base_height" value="0.1673" />
+<xacro:property name="base_height" value="0.1651" />
 <xacro:property name="base_radius" value="0.105" /> <!-- Distance from the motor shaft to the vertical axis -->
 <xacro:property name="imu_offset_z" value="0.063003" />
@@ -15,5 +15,5 @@
 <xacro:property name="wheel_mass" value="0.075" /> <!-- Guesstimate, needs to be measured -->
 <xacro:property name="wheel_thickness" value="0.026" />
-<xacro:property name="base_center_offset_z" value="0.0170" />
+<xacro:property name="base_center_offset_z" value="0.0159" />
 <xacro:property name="footprint_base_offset_z" value="0.085597" /> <!-- CAD offset, Actual offset ~= 0.083597 -->
 <xacro:property name="base_laser_offset_x" value="0.034435" />

Commit message: Update robot.common.xacro

File: urdf/akros2_mecanum/robot.common.xacro (robot description, xacro)
@@ -26,5 +26,5 @@
 <xacro:property name="wheel_mass" value="0.075" /> <!-- Guesstimate, needs to be measured -->
 <xacro:property name="wheel_thickness" value="0.034" /> <!-- Actual thickness = 0.034, CAD thickness = 0.0315 -->
-<xacro:property name="footprint_base_offset_z" value="0.017877" /> <!-- Actual offset = 0.017877, CAD offset = 0.015377 -->
+<xacro:property name="footprint_base_offset_z" value="-0.017877" /> <!-- Actual offset = -0.017877, CAD offset = -0.015377 -->
 <xacro:property name="nav_laser_offset_x" value="0.0632" />
 <xacro:property name="laser_frame_offset_z" value="0.0255" />
