Commit message: remove duplicate frames for IMU

File: urdf/akros2_mecanum/robot.urdf (robot description, URDF)
Before this commit: robot akros2_mecanum, 12 links, 11 joints
Links:
- removed link imu_link
Joints:
- removed joint imu_frame_fixed
- joint imu_base_fixed: child imu_link -> imu_frame

File: urdf/akros2_mecanum/robot.urdf.xacro (robot description, xacro)
@@ -81,6 +81,4 @@
 <link name="laser_frame"/>
 <!-- MPU9250 IMU_LINK -->
-<link name="imu_link"/>
-<!-- IMU_FRAME -->
 <link name="imu_frame"/>
 <!-- WHEEL LEFT FRONT -->
@@ -199,12 +197,6 @@
 <joint name="imu_base_fixed" type="fixed">
   <parent link="base_link"/>
-  <child link="imu_link"/>
+  <child link="imu_frame"/>
   <origin xyz="${imu_offset_x} 0 ${imu_offset_z}"/>
-</joint>
-<!-- IMU_FRAME TO IMU_LINK -->
-<joint name="imu_frame_fixed" type="fixed">
-  <parent link="imu_link"/>
-  <child link="imu_frame"/>
-  <origin xyz="0 0 0"/>
 </joint>
 <!-- WHEEL_LF TO BASE_LINK -->

Commit message: Update robot.urdf

File: urdf/akros2_mecanum/robot.urdf (robot description, URDF)
Before this commit: robot akros2_mecanum, 13 links, 12 joints
Joints:
- removed joint footprint_base_fixed
- added joint base_footprint_fixed: type fixed, parent base_link, child base_footprint, origin xyz=0 0 0.017877

Commit message: Update robot.urdf

File: urdf/akros2_mecanum/robot.urdf (robot description, URDF)
Before this commit: robot akros2_mecanum, 13 links, 12 joints
Joints:
- joint base_footprint_fixed: origin xyz=0 0 0.017877 -> xyz=0 0 -0.017877
