Commit message: remove whitespace

File: urdf/akros2_mecanum/robot.urdf.xacro (robot description, xacro)
@@ -20,5 +20,5 @@
       <mesh filename="${mesh_path}base_module.dae" />
     </geometry>
-   <material name="BaseLinkColor"/>
+    <material name="BaseLinkColor"/>
   </visual>
   <collision>

Commit message: Update robot.urdf.xacro

File: urdf/akros2_mecanum/robot.urdf.xacro (robot description, xacro)
@@ -11,30 +11,30 @@
 </xacro:if>
 <!-- **** LINKS **** -->
+<!-- BASE_LINK -->
+<link name="base_link">
+  <visual>
+    <origin xyz="0 0 0" rpy="0 0 0" />
+    <geometry>
+      <mesh filename="${mesh_path}base_module.dae" />
+    </geometry>
+    <material name="BaseLinkColor"/>
+  </visual>
+  <collision>
+    <origin xyz="${base_offset_x/2} 0 ${base_height/2}" rpy="0 0 0" />
+    <geometry>
+      <box size="${base_length} ${base_width} ${base_height}"/>
+    </geometry>
+  </collision>
+</link>
+<!-- BASE_LINK_INERTIAL (WORKAROUND FOR KDL WHICH DOES NOT ACCEPT BASE_LINK WITH INERTIA) -->
+<link name="base_link_inertial">
+  <inertial>
+    <origin xyz="0 0 0" rpy="0 0 0" />
+    <mass value="${base_mass}"/>
+    <xacro:box_inertia m="${base_mass}" x="${base_length}" y="${base_width}" z="${base_height}"/>
+  </inertial>
+</link>
 <!-- BASE_FOOTPRINT -->
 <link name="base_footprint"/>
-<!-- BASE_LINK -->
-<link name="base_link">
-  <visual>
-    <origin xyz="0 0 0" rpy="0 0 0" />
-    <geometry>
-      <mesh filename="${mesh_path}base_module.dae" />
-    </geometry>
-    <material name="BaseLinkColor"/>
-  </visual>
-  <collision>
-    <origin xyz="${base_offset_x/2} 0 ${base_height/2}" rpy="0 0 0" />
-    <geometry>
-      <box size="${base_length} ${base_width} ${base_height}"/>
-    </geometry>
-  </collision>
-</link>
-<!-- BASE_LINK_INERTIAL (WORKAROUND FOR KDL WHICH DOES NOT ACCEPT BASE_LINK WITH INERTIA) -->
-<link name="base_link_inertial">
-  <inertial>
-    <origin xyz="0 0 0" rpy="0 0 0" />
-    <mass value="${base_mass}"/>
-    <xacro:box_inertia m="${base_mass}" x="${base_length}" y="${base_width}" z="${base_height}"/>
-  </inertial>
-</link>
 <!-- NAV_LINK -->
 <link name="nav_link">
@@ -186,8 +186,8 @@
 </link>
 <!-- **** JOINTS **** -->
-<!-- BASE_LINK TO BASE_FOOTPRINT -->
-<joint name="footprint_base_fixed" type="fixed">
-  <parent link="base_footprint"/>
-  <child link="base_link"/>
+<!-- BASE_FOOTPRINT TO BASE_LINK -->
+<joint name="base_footprint_fixed" type="fixed">
+  <parent link="base_link"/>
+  <child link="base_footprint"/>
   <origin xyz="0 0 ${footprint_base_offset_z}"/>
 </joint>

Commit message: Update robot.urdf.xacro

File: urdf/akros2_mecanum/robot.urdf.xacro (robot description, xacro)
@@ -186,4 +186,10 @@
 </link>
 <!-- **** JOINTS **** -->
+<!-- BASE_LINK_INERTIAL TO BASE_LINK -->
+<joint name="base_inertial_fixed" type="fixed">
+  <parent link="base_link"/>
+  <child link="base_link_inertial"/>
+  <origin xyz="0 0 0"/>
+</joint>
 <!-- BASE_FOOTPRINT TO BASE_LINK -->
 <joint name="base_footprint_fixed" type="fixed">
@@ -191,10 +197,4 @@
   <child link="base_footprint"/>
   <origin xyz="0 0 ${footprint_base_offset_z}"/>
-</joint>
-<!-- BASE_LINK_INERTIAL TO BASE_LINK -->
-<joint name="base_inertial_fixed" type="fixed">
-  <parent link="base_link"/>
-  <child link="base_link_inertial"/>
-  <origin xyz="0 0 0"/>
 </joint>
 <!-- NAV_LINK TO BASE_LINK -->

Commit message: Update robot.urdf.xacro

File: urdf/akros2_mecanum/robot.urdf.xacro (robot description, xacro)
@@ -16,5 +16,5 @@
     <origin xyz="0 0 0" rpy="0 0 0" />
     <geometry>
-      <mesh filename="${mesh_path}base_module.dae" />
+      <mesh filename="${mesh_path}base_module.stl" />
     </geometry>
     <material name="BaseLinkColor"/>
@@ -46,5 +46,5 @@
     <origin xyz="0 0 ${nav_offset_z}" rpy="0 0 0" />
     <geometry>
-      <mesh filename="${mesh_path}navigation_module.dae" />
+      <mesh filename="${mesh_path}navigation_module.stl" />
     </geometry>
     <material name="WheelsNavColor"/>
@@ -67,5 +67,5 @@
     <origin xyz="0 0 0" rpy="0 0 ${-1*pi_by_two}" />
     <geometry>
-      <mesh filename="${mesh_path}ld06.dae" />
+      <mesh filename="${mesh_path}ld06.stl" />
     </geometry>
     <material name="SensorColor"/>
@@ -90,5 +90,5 @@
     <origin xyz="0 0 0" rpy="0 0 0" />
     <geometry>
-      <mesh filename="${mesh_path}cam_module.dae" />
+      <mesh filename="${mesh_path}cam_module.stl" />
     </geometry>
     <material name="SensorColor"/>
@@ -114,5 +114,5 @@
     <origin xyz="0 0 0" rpy="0 0 0" />
     <geometry>
-      <mesh filename="${mesh_path}wheel_lf.dae" />
+      <mesh filename="${mesh_path}wheel_lf.stl" />
     </geometry>
     <material name="WheelsNavColor"/>
@@ -134,5 +134,5 @@
     <origin xyz="0 0 0" rpy="0 0 0" />
     <geometry>
-      <mesh filename="${mesh_path}wheel_lb.dae" />
+      <mesh filename="${mesh_path}wheel_lb.stl" />
     </geometry>
     <material name="WheelsNavColor"/>
@@ -154,5 +154,5 @@
     <origin xyz="0 0 0" rpy="0 0 0" />
     <geometry>
-      <mesh filename="${mesh_path}wheel_rf.dae" />
+      <mesh filename="${mesh_path}wheel_rf.stl" />
     </geometry>
     <material name="WheelsNavColor"/>
@@ -174,5 +174,5 @@
     <origin xyz="0 0 0" rpy="0 0 0" />
     <geometry>
-      <mesh filename="${mesh_path}wheel_rb.dae" />
+      <mesh filename="${mesh_path}wheel_rb.stl" />
     </geometry>
     <material name="WheelsNavColor"/>

Commit message: Update robot.urdf.xacro

File: urdf/akros2_mecanum/robot.urdf.xacro (robot description, xacro)
@@ -4,7 +4,7 @@
 <xacro:include filename="$(find akros2_description)/urdf/akros2_mecanum/robot.control.xacro"/>
 <xacro:include filename="$(find akros2_description)/urdf/akros2_mecanum/robot.gazebo.xacro"/>
-<xacro:arg name="mesh_path" default="package://akros2_description/meshes/akros2_mecanum/" /> <!-- HTTPS URL also works here -->
+<xacro:arg name="mesh_path_mecanum" default="package://akros2_description/meshes/akros2_mecanum/" /> <!-- HTTPS URL also works here -->
 <xacro:arg name="nopath" default="false" />
-<xacro:property name="mesh_path" value="$(arg mesh_path)" />
+<xacro:property name="mesh_path" value="$(arg mesh_path_mecanum)" />
 <xacro:if value="$(arg nopath)">
   <xacro:property name="mesh_path" value="" />
