Commit message: Update robot.gazebo.xacro

File: urdf/akros2_diff/robot.gazebo.xacro (robot description, xacro)
@@ -3,10 +3,4 @@
 <gazebo reference="base_link">
   <material>Gazebo/Grey</material>
-</gazebo>
-<gazebo reference="laser_link">
-  <material>Gazebo/FlatBlack</material>
-</gazebo>
-<gazebo reference="wheel_f">
-  <material>Gazebo/DarkGrey</material>
 </gazebo>
 <gazebo reference="wheel_l">
@@ -15,35 +9,4 @@
 <gazebo reference="wheel_r">
   <material>Gazebo/DarkGrey</material>
-</gazebo>
-<gazebo reference="laser_frame">
-  <sensor type="ray" name="head_ld06_sensor">
-    <pose>0 0 0.06 0 0 0</pose>
-    <visualize>false</visualize>
-    <update_rate>40</update_rate>
-    <ray>
-      <scan>
-        <horizontal>
-          <samples>720</samples>
-          <resolution>1</resolution>
-          <min_angle>-3.14159265</min_angle>
-          <max_angle>3.14159265</max_angle>
-        </horizontal>
-      </scan>
-      <range>
-        <min>0.2</min>
-        <max>30.0</max>
-        <resolution>0.01</resolution>
-      </range>
-      <noise>
-        <type>gaussian</type>
-        <mean>0.0</mean>
-        <stddev>0.01</stddev>
-      </noise>
-    </ray>
-    <plugin name="gazebo_ros_head_ld06_controller" filename="libgazebo_ros_laser.so">
-      <topicName>scan</topicName>
-      <frameName>laser_frame</frameName>
-    </plugin>
-  </sensor>
 </gazebo>
 <gazebo>
@@ -76,5 +39,5 @@
 </gazebo>
 <gazebo>
-  <plugin name="omni_steering" filename="libgazebo_ros_planar_move.so">
+  <plugin name="diff_steering" filename="libgazebo_ros_planar_move.so">
     <commandTopic>cmd_vel</commandTopic>
     <odometryTopic>odom</odometryTopic>
