Commit message: update urdfs

File: urdf/akros2_diff/robot.common.xacro (robot description, xacro)
@@ -1,15 +1,10 @@
 <?xml version="1.0" encoding="utf-8"?>
-<robot name="omni_common" xmlns:xacro="http://ros.org/wiki/xacro">
+<robot name="diff_common" xmlns:xacro="http://ros.org/wiki/xacro">
 <!-- All values below are based on the CAD model (Fusion 360) -->
 <xacro:property name="pi_by_two" value="1.5707963" />
-<xacro:property name="pi_by_three" value="1.0471975"/>
 <xacro:property name="base_mass" value="2.0" /> <!-- Guesstimate, needs to be measured -->
 <xacro:property name="base_height" value="0.1651" />
 <xacro:property name="base_radius" value="0.105" /> <!-- Distance from the motor shaft to the vertical axis -->
 <xacro:property name="imu_offset_z" value="0.063003" />
-<xacro:property name="laser_mass" value="0.12" />
-<xacro:property name="laser_length" value="0.038" />
-<xacro:property name="laser_width" value="0.0381" />
-<xacro:property name="laser_height" value="0.033" />
 <xacro:property name="wheel_radius" value="0.029" />
 <xacro:property name="wheel_mass" value="0.075" /> <!-- Guesstimate, needs to be measured -->
@@ -17,8 +12,4 @@
 <xacro:property name="base_center_offset_z" value="0.0164" />
 <xacro:property name="footprint_base_offset_z" value="0.085597" /> <!-- CAD offset, Actual offset ~= 0.083597 -->
-<xacro:property name="base_laser_offset_x" value="0.034435" />
-<xacro:property name="base_laser_offset_z" value="0.076503" />
-<xacro:property name="laser_frame_offset_z" value="0.0255" />
-<xacro:property name="joint_f_offset_x" value="0.10683" />
 <xacro:property name="joint_lr_offset_x" value="-0.053415" />
 <xacro:property name="joint_lr_offset_y" value="0.092518" />
@@ -39,7 +30,4 @@
             izz="${2*m*r*r/5}" />
 </xacro:macro>
-<material name="LaserColor">
-    <color rgba="0.2 0.2 0.2 1"/>
-</material>
 <material name="WheelsNavColor">
     <color rgba="0.35 0.35 0.35 1"/>

File: urdf/akros2_diff/robot.gazebo.xacro (robot description, xacro)
@@ -1,4 +1,4 @@
 <?xml version="1.0" encoding="utf-8"?>
-<robot name="omni_gazebo" xmlns:xacro="http://ros.org/wiki/xacro">
+<robot name="diff_gazebo" xmlns:xacro="http://ros.org/wiki/xacro">
 <gazebo reference="base_link">
   <material>Gazebo/Grey</material>

File: urdf/akros2_diff/robot.urdf (robot description, URDF)
Before this commit: robot akros2_omni, 9 links, 8 joints
Links:
- removed link laser_frame
- removed link laser_link
- removed link wheel_f
- link base_link: geometry collision cylinder length=0.1651 radius=0.105; visual mesh filename=package://akros2_description/meshes/akros2_diff/base_module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
- link wheel_l: geometry collision cylinder length=0.026 radius=0.029; visual mesh filename=package://akros2_description/meshes/akros2_diff/omniwheel.d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
- link wheel_r: geometry collision cylinder length=0.026 radius=0.029; visual mesh filename=package://akros2_description/meshes/akros2_diff/omniwheel.d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
Joints:
- removed joint base_laser_fixed
- removed joint joint_f
- removed joint laser_frame_fixed
