Commit message: Update robot.urdf

File: urdf/akros2_diff/robot.urdf (robot description, URDF)
Before this commit: robot akros2_omni, 9 links, 8 joints
Joints:
- removed joint footprint_base_fixed
- added joint base_footprint_fixed: type fixed, parent base_link, child base_footprint, origin xyz=0 0 0.085597

Commit message: update .dae to .stl

File: urdf/akros2_diff/robot.urdf (robot description, URDF)
Before this commit: robot akros2_diff, 6 links, 5 joints
Links:
- link wheel_l: geometry collision cylinder length=0.026 radius=0.029; visual mesh filename=package://akros2_description/meshes/akros2_diff/wheel.stl
- link wheel_r: geometry collision cylinder length=0.026 radius=0.029; visual mesh filename=package://akros2_description/meshes/akros2_diff/wheel.stl

File: urdf/akros2_diff/robot.urdf.xacro (robot description, xacro)
@@ -16,5 +16,5 @@
     <origin xyz="0 0 0" rpy="0 0 0" />
     <geometry>
-      <mesh filename="${mesh_path}base_module.dae" />
+      <mesh filename="${mesh_path}base_module.stl" />
     </geometry>
     <material name="BaseLinkColor"/>
@@ -48,5 +48,5 @@
     <origin xyz="0 0 0" rpy="0 0 0" />
     <geometry>
-      <mesh filename="${mesh_path}wheel.dae" />
+      <mesh filename="${mesh_path}wheel.stl" />
     </geometry>
     <material name="WheelsNavColor"/>
@@ -68,5 +68,5 @@
     <origin xyz="0 0 0" rpy="0 0 0" />
     <geometry>
-      <mesh filename="${mesh_path}wheel.dae" />
+      <mesh filename="${mesh_path}wheel.stl" />
     </geometry>
     <material name="WheelsNavColor"/>

File: urdf/akros2_mecanum/robot.urdf (robot description, URDF)
Before this commit: robot akros2_mecanum, 13 links, 12 joints
Links:
- link laser_link: geometry collision box size=0.042 0.0421 0.033; visual mesh filename=package://akros2_description/meshes/akros2_mecanum/ld06.stl

File: urdf/akros2_omni/robot.urdf (robot description, URDF)
Before this commit: robot akros2_omni, 9 links, 8 joints
Links:
- link laser_link: geometry collision box size=0.038 0.0381 0.033; visual mesh filename=package://akros2_description/meshes/akros2_omni/ld06.stl
- link wheel_f: geometry collision cylinder length=0.026 radius=0.029; visual mesh filename=package://akros2_description/meshes/akros2_omni/omniwheel.s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
- link wheel_l: geometry collision cylinder length=0.026 radius=0.029; visual mesh filename=package://akros2_description/meshes/akros2_omni/omniwheel.s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
- link wheel_r: geometry collision cylinder length=0.026 radius=0.029; visual mesh filename=package://akros2_description/meshes/akros2_omni/omniwheel.s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

File: urdf/akros2_omni/robot.urdf.xacro (robot description, xacro)
@@ -16,5 +16,5 @@
     <origin xyz="0 0 0" rpy="0 0 0" />
     <geometry>
-      <mesh filename="${mesh_path}base_module.dae" />
+      <mesh filename="${mesh_path}base_module.stl" />
     </geometry>
     <material name="BaseLinkColor"/>
@@ -47,5 +47,5 @@
     <origin xyz="0 0 0" rpy="0 0 ${-1*pi_by_two}" />
     <geometry>
-      <mesh filename="${mesh_path}ld06.dae" />
+      <mesh filename="${mesh_path}ld06.stl" />
     </geometry>
     <material name="LaserColor"/>
@@ -71,5 +71,5 @@
     <origin xyz="0 0 0" rpy="0 0 0" />
     <geometry>
-      <mesh filename="${mesh_path}omniwheel.dae" />
+      <mesh filename="${mesh_path}omniwheel.stl" />
     </geometry>
     <material name="WheelsNavColor"/>
@@ -91,5 +91,5 @@
     <origin xyz="0 0 0" rpy="0 0 0" />
     <geometry>
-      <mesh filename="${mesh_path}omniwheel.dae" />
+      <mesh filename="${mesh_path}omniwheel.stl" />
     </geometry>
     <material name="WheelsNavColor"/>
@@ -111,5 +111,5 @@
     <origin xyz="0 0 0" rpy="0 0 0" />
     <geometry>
-      <mesh filename="${mesh_path}omniwheel.dae" />
+      <mesh filename="${mesh_path}omniwheel.stl" />
     </geometry>
     <material name="WheelsNavColor"/>
