Commit message: Update robot.urdf

File: urdf/akros2_omni/robot.urdf (robot description, URDF)
Before this commit: robot akros2_omni, 9 links, 8 joints
Joints:
- removed joint footprint_base_fixed
- added joint base_footprint_fixed: type fixed, parent base_link, child base_footprint, origin xyz=0 0 -0.085597
