Commit message: added akros2_omni urdf, updated meshes

File: urdf/akros2_omni/robot.urdf.xacro (robot description, xacro)
@@ -5,7 +5,7 @@
 <xacro:include filename="$(find akros2_description)/urdf/akros2_omni/robot.gazebo.xacro"/>
 <xacro:arg name="mesh_path" default="package://akros2_description/meshes/akros2_omni/" /> <!-- HTTPS URL also works here -->
-<xacro:arg name="unity" default="false" />
+<xacro:arg name="nopath" default="false" />
 <xacro:property name="mesh_path" value="$(arg mesh_path)" />
-<xacro:if value="$(arg unity)">
+<xacro:if value="$(arg nopath)">
   <xacro:property name="mesh_path" value="" />
 </xacro:if>

File: urdf/akros2_omni/robot2.urdf (robot description, URDF)
Before this commit: robot akros2_omni, 9 links, 8 joints
Links:
- link base_link: geometry collision cylinder length=0.1651 radius=0.105; visual mesh filename=base_module.dae
- link laser_link: geometry collision box size=0.038 0.0381 0.033; visual mesh filename=ld06.dae
- link wheel_f: geometry collision cylinder length=0.026 radius=0.029; visual mesh filename=omniwheel.dae
- link wheel_l: geometry collision cylinder length=0.026 radius=0.029; visual mesh filename=omniwheel.dae
- link wheel_r: geometry collision cylinder length=0.026 radius=0.029; visual mesh filename=omniwheel.dae

Commit message: Update robot.urdf.xacro

File: urdf/akros2_omni/robot.urdf.xacro (robot description, xacro)
@@ -11,6 +11,4 @@
 </xacro:if>
 <!-- **** LINKS **** -->
-<!-- BASE_FOOTPRINT -->
-<link name="base_footprint"/>
 <!-- BASE_LINK -->
 <link name="base_link">
@@ -37,4 +35,6 @@
   </inertial>
 </link>
+<!-- BASE_FOOTPRINT -->
+<link name="base_footprint"/>
 <!-- LD06 LASER_LINK -->
 <link name="laser_link">
@@ -60,5 +60,5 @@
 <!-- LASER_FRAME -->
 <link name="laser_frame"/>
-<!-- MPU9250 IMU_LINK -->
+<!-- BNO085 IMU_LINK -->
 <link name="imu_link"/>
 <!-- WHEEL FRONT -->
@@ -123,10 +123,4 @@
 </link>
 <!-- **** JOINTS **** -->
-<!-- BASE_LINK TO BASE_FOOTPRINT -->
-<joint name="footprint_base_fixed" type="fixed">
-  <parent link="base_footprint"/>
-  <child link="base_link"/>
-  <origin xyz="0 0 ${footprint_base_offset_z}"/>
-</joint>
 <!-- BASE_LINK_INERTIAL TO BASE_LINK -->
 <joint name="base_inertial_fixed" type="fixed">
@@ -134,4 +128,10 @@
   <child link="base_link_inertial"/>
   <origin xyz="0 0 0"/>
+</joint>
+<!-- BASE_FOOTPRINT TO BASE_LINK -->
+<joint name="base_footprint_fixed" type="fixed">
+  <parent link="base_link"/>
+  <child link="base_footprint"/>
+  <origin xyz="0 0 ${footprint_base_offset_z}"/>
 </joint>
 <!-- LASER_LINK TO BASE_LINK -->

Commit message: Update robot.urdf.xacro

File: urdf/akros2_omni/robot.urdf.xacro (robot description, xacro)
@@ -4,7 +4,7 @@
 <xacro:include filename="$(find akros2_description)/urdf/akros2_omni/robot.control.xacro"/>
 <xacro:include filename="$(find akros2_description)/urdf/akros2_omni/robot.gazebo.xacro"/>
-<xacro:arg name="mesh_path" default="package://akros2_description/meshes/akros2_omni/" /> <!-- HTTPS URL also works here -->
+<xacro:arg name="mesh_path_omni" default="package://akros2_description/meshes/akros2_omni/" /> <!-- HTTPS URL also works here -->
 <xacro:arg name="nopath" default="false" />
-<xacro:property name="mesh_path" value="$(arg mesh_path)" />
+<xacro:property name="mesh_path" value="$(arg mesh_path_omni)" />
 <xacro:if value="$(arg nopath)">
   <xacro:property name="mesh_path" value="" />
